Commit message: urdf file geometries are now correct and functional, still can't load stl's into rviz

File: src/surg_bot/surg_bot_description/urdf/surg_bot_description.urdf (robot description, URDF)
Before this commit: robot surg_bot_description, 5 links, 4 joints
Links:
- removed link Base
- added link base_link, mass 15.865948579379; collision mesh filename=package://surg_bot_description/meshes/Base.stl; visual mesh filename=package://surg_bot_description/meshes/Base.stl
- added link world
- link Link1: geometry collision mesh filename=package://surg_bot_description/meshes/Link1.stl; visual mesh filename=package://surg_bot_description/meshes/Link1.stl
- link Link2: geometry collision mesh filename=package://surg_bot_description/meshes/Link2.stl; visual mesh filename=package://surg_bot_description/meshes/Link2.stl
- link Link3: geometry collision mesh filename=package://surg_bot_description/meshes/Link3.stl; visual mesh filename=package://surg_bot_description/meshes/Link3.stl
- link Link4: geometry collision mesh filename=package://surg_bot_description/meshes/Link4.stl; visual mesh filename=package://surg_bot_description/meshes/Link4.stl
Joints:
- added joint world_to_base_link=: type fixed, parent world, child base_link
- joint Joint0: parent Base -> base_link

Commit message: Deleted Even more unnecessary files

File: src/surg_bot/surg_bot_description/urdf/surg_bot_description.urdf (robot description, URDF)
Before this commit: robot surg_bot_description, 6 links, 5 joints
Links:
- removed link base_link
- removed link world
- added link Base, mass 15.865948579379; collision mesh filename=package://surg_bot_description/meshes/Base.STL; visual mesh filename=package://surg_bot_description/meshes/Base.STL
- added link Link5, mass 0.283181051897044; collision mesh filename=package://surg_bot_description/meshes/Link5.STL; visual mesh filename=package://surg_bot_description/meshes/Link5.STL
- added link Link6, mass 0.467880622236969; collision mesh filename=package://surg_bot_description/meshes/Link6.STL; visual mesh filename=package://surg_bot_description/meshes/Link6.STL
- added link Link7, mass 1.16594380268497; collision mesh filename=package://surg_bot_description/meshes/Link7.STL; visual mesh filename=package://surg_bot_description/meshes/Link7.STL
- added link Link8, mass 44.0763599099016; collision mesh filename=package://surg_bot_description/meshes/Link8.STL; visual mesh filename=package://surg_bot_description/meshes/Link8.STL
- link Link1: geometry collision mesh filename=package://surg_bot_description/meshes/Link1.STL; visual mesh filename=package://surg_bot_description/meshes/Link1.STL
- link Link2: geometry collision mesh filename=package://surg_bot_description/meshes/Link2.STL; visual mesh filename=package://surg_bot_description/meshes/Link2.STL
- link Link3: mass 1.24438737439991 -> 1.2443873743999; geometry collision mesh filename=package://surg_bot_description/meshes/Link3.STL; visual mesh filename=package://surg_bot_description/meshes/Link3.STL
- link Link4: mass 4.30755194902526 -> 4.09760403890471; geometry collision mesh filename=package://surg_bot_description/meshes/Link4.STL; visual mesh filename=package://surg_bot_description/meshes/Link4.STL
Joints:
- removed joint Joint0
- removed joint Joint1
- removed joint Joint2
- removed joint Joint3
- removed joint world_to_base_link=
- added joint Link1: type revolute, parent Base, child Link1, origin xyz=0 0 0 rpy=0 0 0, axis 0 1 0, limit lower=0 upper=0 effort=10 velocity=10
- added joint Link2: type revolute, parent Base, child Link2, origin xyz=0 0 0 rpy=0 0 0, axis 0 -1 0, limit lower=0 upper=0 effort=10 velocity=10
- added joint Link3: type revolute, parent Base, child Link3, origin xyz=0 0 0 rpy=0 0 0, axis 0 0 1, limit lower=0 upper=0 effort=10 velocity=10
- added joint Link4: type revolute, parent Base, child Link4, origin xyz=0 0 0 rpy=0 0 0, axis 0 0 1, limit lower=0 upper=0 effort=10 velocity=10
- added joint Link5: type revolute, parent Base, child Link5, origin xyz=0 0 0 rpy=0 0 0, axis -1 0 0, limit lower=0 upper=0 effort=10 velocity=10
- added joint Link6: type revolute, parent Base, child Link6, origin xyz=0 0 0 rpy=0 0 0, axis -1 0 0, limit lower=0 upper=0 effort=10 velocity=10
- added joint Link7: type revolute, parent Base, child Link7, origin xyz=0 0 0 rpy=0 0 0, axis -1 0 0, limit lower=0 upper=0 effort=10 velocity=10
- added joint Link8: type revolute, parent Base, child Link8, origin xyz=0 0 0 rpy=0 0 0, axis 0 0 -1, limit lower=0 upper=0 effort=10 velocity=10
