Commit message: The URDF is like actually good, like joint states and everything

File: ros2_ws/src/surg_bot/surg_bot_gazebo/urdf/surg_bot_gazebo.urdf (robot description, URDF)
Before this commit: robot surg_bot_description, 10 links, 9 joints
Links:
- removed link dummy
- link Lamp: geometry collision mesh filename=../meshes/Lamp.STL; visual mesh filename=../meshes/Lamp.STL
- link Link1: geometry collision mesh filename=../meshes/Link1.STL; visual mesh filename=../meshes/Link1.STL
- link Link2: geometry collision mesh filename=../meshes/Link2.STL; visual mesh filename=../meshes/Link2.STL
- link Link3: geometry collision mesh filename=../meshes/Link3.STL; visual mesh filename=../meshes/Link3.STL
- link Link4: geometry collision mesh filename=../meshes/Link4.STL; visual mesh filename=../meshes/Link4.STL
- link Link5: geometry collision mesh filename=../meshes/Link5.STL; visual mesh filename=../meshes/Link5.STL
- link Link6: geometry collision mesh filename=../meshes/Link6.STL; visual mesh filename=../meshes/Link6.STL
- link Link7: geometry collision mesh filename=../meshes/Link7.STL; visual mesh filename=../meshes/Link7.STL
- link base_link: geometry collision mesh filename=../meshes/base_link.STL; visual mesh filename=../meshes/base_link.STL
Joints:
- removed joint dummy_joint
- joint Joint0: type continuous -> revolute
- joint Joint1: type continuous -> revolute
- joint Joint2: origin xyz=-0.0508 1.6976E-07 0 rpy=0 0 0 -> xyz=-0.0508 0.127 0 rpy=0 0 0
- joint Joint3: type fixed -> continuous
- joint Joint4: type fixed -> revolute
- joint Joint6: type fixed -> continuous
- joint Joint7: type continuous -> revolute
