Commit message: Changed naming conventions

File: ros2_ws/surg_bot/surg_bot_description/urdf/surg_bot_description.urdf (robot description, URDF)
Before this commit: robot surg_bot_description, 10 links, 9 joints
Joints:
- joint Joint0: origin xyz=0.10643 -0.19117 0 rpy=1.5708 0 0 -> xyz=0 0 0 rpy=1.5708 0 0
- joint ceiling_joint: origin (none) -> xyz=0 0 -0.2 rpy=0 0 0
