Commit message: Added python package for the hand tracking algorithm

File: ros2_ws/src/surg_bot/surg_bot_description/urdf/surg_bot_description.urdf (robot description, URDF)
Before this commit: robot surg_bot_description, 9 links, 8 joints
Links:
- removed link Base
- added link base_link, mass 15.865948579379; collision mesh filename=package://surg_bot_description/meshes/Base.STL; visual mesh filename=package://surg_bot_description/meshes/Base.STL
- added link dummy_link, mass 0
- link Link1: mass 7.06121044359283 -> 7.06121044359282
- link Link8: mass 44.0763599099016 -> 75.3932063564624
Joints:
- added joint dummy_joint: type fixed, parent dummy_link, child base_link, origin xyz=0 0 0
- joint Link1: limit lower=0 upper=0 effort=10 velocity=10 -> lower=0 upper=360 effort=10 velocity=10
- joint Link2: limit lower=0 upper=0 effort=10 velocity=10 -> lower=0 upper=360 effort=10 velocity=10; parent Base -> Link1
- joint Link3: limit lower=0 upper=0 effort=10 velocity=10 -> lower=0 upper=360 effort=10 velocity=10; parent Base -> Link2
- joint Link4: limit lower=0 upper=0 effort=10 velocity=10 -> lower=0 upper=360 effort=10 velocity=10; parent Base -> Link3
- joint Link5: limit lower=0 upper=0 effort=10 velocity=10 -> lower=0 upper=360 effort=10 velocity=10; parent Base -> Link4
- joint Link6: limit lower=0 upper=0 effort=10 velocity=10 -> lower=0 upper=360 effort=10 velocity=10; parent Base -> Link5
- joint Link7: limit lower=0 upper=0 effort=10 velocity=10 -> lower=0 upper=360 effort=10 velocity=10; parent Base -> Link6
- joint Link8: limit lower=0 upper=0 effort=10 velocity=10 -> lower=0 upper=360 effort=10 velocity=10; parent Base -> Link7

Commit message: I did a lot of stuff, but the URDF should be chill

File: ros2_ws/src/surg_bot/surg_bot_description/urdf/surg_bot_description.urdf (robot description, URDF)
Before this commit: robot surg_bot_description, 10 links, 9 joints
Links:
- removed link base_link
- removed link dummy_link
- added link Base, mass 15.865948579379; collision mesh filename=package://test_urdf_tool/meshes/visual/Base.STL; visual mesh filename=package://test_urdf_tool/meshes/visual/Base.STL
- added link base_footprint; visual box size=0.001 0.001 0.001
- link Link1: geometry collision mesh filename=package://test_urdf_tool/meshes/visual/Link1.STL; visual mesh filename=package://test_urdf_tool/meshes/visual/Link1.STL
- link Link2: geometry collision mesh filename=package://test_urdf_tool/meshes/visual/Link2.STL; visual mesh filename=package://test_urdf_tool/meshes/visual/Link2.STL
- link Link3: geometry collision mesh filename=package://test_urdf_tool/meshes/visual/Link3.STL; visual mesh filename=package://test_urdf_tool/meshes/visual/Link3.STL
- link Link4: geometry collision mesh filename=package://test_urdf_tool/meshes/visual/Link4.STL; visual mesh filename=package://test_urdf_tool/meshes/visual/Link4.STL
- link Link5: geometry collision mesh filename=package://test_urdf_tool/meshes/visual/Link5.STL; visual mesh filename=package://test_urdf_tool/meshes/visual/Link5.STL
- link Link6: geometry collision mesh filename=package://test_urdf_tool/meshes/visual/Link6.STL; visual mesh filename=package://test_urdf_tool/meshes/visual/Link6.STL
- link Link7: geometry collision mesh filename=package://test_urdf_tool/meshes/visual/Link7.STL; visual mesh filename=package://test_urdf_tool/meshes/visual/Link7.STL
- link Link8: geometry collision mesh filename=package://test_urdf_tool/meshes/visual/Link8.STL; visual mesh filename=package://test_urdf_tool/meshes/visual/Link8.STL
Joints:
- removed joint dummy_joint
- added joint base_footprint_joint: type fixed, parent base_footprint, child base_link, origin xyz=0 0 0.001 rpy=0 0 0

Commit message: Have a functioning URDF now, converted it to SDF for Gazebo use URDF import still a little wonky, need to export a new one from solidworks

File: ros2_ws/src/surg_bot/surg_bot_description/urdf/surg_bot_description.urdf (robot description, URDF)
Before this commit: robot surg_bot_description, 10 links, 9 joints
Links:
- removed link Base
- removed link Link8
- removed link base_footprint
- added link Lamp, mass 44.076; collision mesh filename=../meshes/Lamp.STL; visual mesh filename=../meshes/Lamp.STL
- added link base_link, mass 15.865948579379; collision mesh filename=../meshes/base_link.STL; visual mesh filename=../meshes/base_link.STL
- link Link1: mass 7.06121044359282 -> 7.0612; geometry collision mesh filename=../meshes/Link1.STL; visual mesh filename=../meshes/Link1.STL
- link Link2: mass 1.13069874193925 -> 1.1307; geometry collision mesh filename=../meshes/Link2.STL; visual mesh filename=../meshes/Link2.STL
- link Link3: mass 1.2443873743999 -> 1.2444; geometry collision mesh filename=../meshes/Link3.STL; visual mesh filename=../meshes/Link3.STL
- link Link4: mass 4.09760403890471 -> 4.0976; geometry collision mesh filename=../meshes/Link4.STL; visual mesh filename=../meshes/Link4.STL
- link Link5: mass 0.283181051897044 -> 0.28318; geometry collision mesh filename=../meshes/Link5.STL; visual mesh filename=../meshes/Link5.STL
- link Link6: mass 0.467880622236969 -> 0.46788; geometry collision mesh filename=../meshes/Link6.STL; visual mesh filename=../meshes/Link6.STL
- link Link7: mass 1.16594380268497 -> 1.1659; geometry collision mesh filename=../meshes/Link7.STL; visual mesh filename=../meshes/Link7.STL
Joints:
- removed joint Link1
- removed joint Link2
- removed joint Link3
- removed joint Link4
- removed joint Link5
- removed joint Link6
- removed joint Link7
- removed joint Link8
- removed joint base_footprint_joint
- added joint Joint0: type revolute, parent base_link, child Link1, origin xyz=0.10643 -0.19117 0 rpy=1.5708 0 0, axis 0 1 0, limit lower=0 upper=0 effort=0 velocity=0
- added joint Joint1: type revolute, parent Link1, child Link2, origin xyz=0.8636 -0.37436 0 rpy=0 -1.5708 0, axis 0 1 0, limit lower=0 upper=0 effort=0 velocity=0
- added joint Joint2: type continuous, parent Link2, child Link3, origin xyz=-0.0508 0.127 0 rpy=0 0 0, axis 1 0 0
- added joint Joint3: type continuous, parent Link3, child Link4, origin xyz=-0.0762 0 -0.0508 rpy=0 0 3.1416, axis 0 0 1
- added joint Joint4: type revolute, parent Link4, child Link5, origin xyz=0 0 -0.8382 rpy=0 0 3.1416, axis 0 0 1, limit lower=0 upper=0 effort=0 velocity=0
- added joint Joint5: type continuous, parent Link5, child Link6, origin xyz=0 0.01 0 rpy=0 0 0, axis 0 0 1
- added joint Joint6: type continuous, parent Link6, child Link7, origin xyz=0.34214 -0.028375 -0.41803 rpy=0 0 3.1416, axis 0 0 1
- added joint Joint7: type revolute, parent Link7, child Lamp, origin xyz=0.044276 -0.018375 -0.014756 rpy=0 0 0, axis 1 0 0, limit lower=0 upper=0 effort=0 velocity=0

Commit message: Testing

File: ros2_ws/src/surg_bot/surg_bot_description/urdf/surg_bot_description.urdf (robot description, URDF)
Before this commit: robot surg_bot_description, 10 links, 9 joints
Links:
- removed link dummy
- added link ceiling; visual box size=1 1 0.1
Joints:
- removed joint dummy_joint
- added joint ceiling_joint: type fixed, parent ceiling, child base_link

File: ros2_ws/src/surg_bot/surg_bot_gazebo/urdf/surg_bot_description.urdf (robot description, URDF)
Before this commit: robot surg_bot_description, 9 links, 8 joints
Links:
- added link ceiling; visual box size=1 1 0.1
- link Lamp: geometry collision mesh filename=/home/alec/Autotracking_Surgical_Lamp/ros2_ws/src/surg_bot/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; visual mesh filename=/home/alec/Autotracking_Surgical_Lamp/ros2_ws/src/surg_bot/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
- link Link1: geometry collision mesh filename=/home/alec/Autotracking_Surgical_Lamp/ros2_ws/src/surg_bot/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; visual mesh filename=/home/alec/Autotracking_Surgical_Lamp/ros2_ws/src/surg_bot/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
- link Link2: geometry collision mesh filename=/home/alec/Autotracking_Surgical_Lamp/ros2_ws/src/surg_bot/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; visual mesh filename=/home/alec/Autotracking_Surgical_Lamp/ros2_ws/src/surg_bot/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
- link Link3: geometry collision mesh filename=/home/alec/Autotracking_Surgical_Lamp/ros2_ws/src/surg_bot/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; visual mesh filename=/home/alec/Autotracking_Surgical_Lamp/ros2_ws/src/surg_bot/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
- link Link4: geometry collision mesh filename=/home/alec/Autotracking_Surgical_Lamp/ros2_ws/src/surg_bot/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; visual mesh filename=/home/alec/Autotracking_Surgical_Lamp/ros2_ws/src/surg_bot/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
- link Link5: geometry collision mesh filename=/home/alec/Autotracking_Surgical_Lamp/ros2_ws/src/surg_bot/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; visual mesh filename=/home/alec/Autotracking_Surgical_Lamp/ros2_ws/src/surg_bot/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
- link Link6: geometry collision mesh filename=/home/alec/Autotracking_Surgical_Lamp/ros2_ws/src/surg_bot/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; visual mesh filename=/home/alec/Autotracking_Surgical_Lamp/ros2_ws/src/surg_bot/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
- link Link7: geometry collision mesh filename=/home/alec/Autotracking_Surgical_Lamp/ros2_ws/src/surg_bot/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; visual mesh filename=/home/alec/Autotracking_Surgical_Lamp/ros2_ws/src/surg_bot/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
- link base_link: geometry collision mesh filename=/home/alec/Autotracking_Surgical_Lamp/ros2_ws/src/surg_bot/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; visual mesh filename=/home/alec/Autotracking_Surgical_Lamp/ros2_ws/src/surg_bot/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
Joints:
- added joint ceiling_joint: type fixed, parent ceiling, child base_link
- joint Joint0: type revolute -> continuous
- joint Joint1: type revolute -> continuous
- joint Joint2: origin xyz=-0.0508 0.127 0 rpy=0 0 0 -> xyz=-0.0508 1.6976E-07 0 rpy=0 0 0
- joint Joint3: type continuous -> fixed
- joint Joint4: type revolute -> fixed
- joint Joint6: type continuous -> fixed
- joint Joint7: type revolute -> continuous

Commit message: idk

File: ros2_ws/src/surg_bot/surg_bot_description/urdf/surg_bot_description.urdf (robot description, URDF)
Before this commit: robot surg_bot_description, 10 links, 9 joints
Joints:
- joint ceiling_joint: origin xyz=0 0 -0.2 rpy=0 0 0 -> xyz=0 0 -0.37 rpy=0 0 0

Commit message: Meshes are working in RVIZ but URDF needs to be completely reworked

File: ros2_ws/src/surg_bot/surg_bot_description/urdf/surg_bot_description.urdf (robot description, URDF)
Before this commit: robot surg_bot_description, 10 links, 9 joints
Links:
- removed link Link1
- removed link Link2
- removed link Link3
- removed link Link4
- removed link Link5
- removed link Link6
- removed link Link7
- added link link1, mass 7.0612; collision mesh filename=file://$(find surg_bot_description)/meshes/link1.dae; visual mesh filename=file://$(find surg_bot_description)/meshes/link1.dae
- added link link2, mass 1.1307; collision mesh filename=file://$(find surg_bot_description)/meshes/link2.dae; visual mesh filename=file://$(find surg_bot_description)/meshes/link2.dae
- added link link3, mass 1.2444; collision mesh filename=file://$(find surg_bot_description)/meshes/link3.dae; visual mesh filename=file://$(find surg_bot_description)/meshes/link3.dae
- added link link4, mass 4.0976; collision mesh filename=file://$(find surg_bot_description)/meshes/link4.dae; visual mesh filename=file://$(find surg_bot_description)/meshes/link4.dae
- added link link5, mass 0.28318; collision mesh filename=file://$(find surg_bot_description)/meshes/link5.dae; visual mesh filename=file://$(find surg_bot_description)/meshes/link5.dae
- added link link6, mass 0.46788; collision mesh filename=file://$(find surg_bot_description)/meshes/link6.dae; visual mesh filename=file://$(find surg_bot_description)/meshes/link6.dae
- added link link7, mass 1.1659; collision mesh filename=file://$(find surg_bot_description)/meshes/link7.dae; visual mesh filename=file://$(find surg_bot_description)/meshes/link7.dae
- link Lamp: geometry collision mesh filename=file://$(find surg_bot_description)/meshes/lamp.dae; visual mesh filename=file://$(find surg_bot_description)/meshes/lamp.dae
- link base_link: geometry collision mesh filename=file://$(find surg_bot_description)/meshes/base_link.dae; visual mesh filename=file://$(find surg_bot_description)/meshes/base_link.dae
Joints:
- joint Joint0: axis 0 1 0 -> 0 0 1; child Link1 -> link1; origin xyz=0 0 0 rpy=1.5708 0 0 -> xyz=0 0 0 rpy=0 0 1.5708
- joint Joint1: child Link2 -> link2; parent Link1 -> link1
- joint Joint2: child Link3 -> link3; parent Link2 -> link2
- joint Joint3: child Link4 -> link4; parent Link3 -> link3
- joint Joint4: child Link5 -> link5; parent Link4 -> link4
- joint Joint5: child Link6 -> link6; parent Link5 -> link5
- joint Joint6: child Link7 -> link7; parent Link6 -> link6
- joint Joint7: parent Link7 -> link7
- joint ceiling_joint: origin xyz=0 0 -0.37 rpy=0 0 0 -> xyz=0 0 -.37 rpy=0 0 0

Commit message: The URDF is like actually finally perfect for realsies this time

File: ros2_ws/src/surg_bot/surg_bot_description/urdf/surg_bot_description.urdf (robot description, URDF)
Before this commit: robot surg_bot_description, 10 links, 9 joints
Joints:
- joint Joint0: origin xyz=0 0 0 rpy=0 0 1.5708 -> xyz=0 0 -0.445 rpy=0 0 0
- joint Joint1: axis 0 1 0 -> 0 0 1; origin xyz=0.8636 -0.37436 0 rpy=0 -1.5708 0 -> xyz=0.8636 0 -0.28 rpy=0 0 1.57
- joint Joint2: origin xyz=-0.0508 1.6976E-07 0 rpy=0 0 0 -> xyz=-0.064 0 -0.127  rpy=1.57 0 0
- joint Joint3: origin xyz=-0.0762 0 -0.0508 rpy=0 0 3.1416 -> xyz=-0.0762 0 -0.127 rpy=0 0 3.1416
- joint Joint4: origin xyz=0 0 -0.8382 rpy=0 0 3.1416 -> xyz=0 0 -0.762 rpy=0 0 3.1416; type fixed -> continuous
- joint Joint5: origin xyz=0 0.01 0 rpy=0 0 0 -> xyz=0.05 0 -0.067 rpy=0 -1.57 0; type continuous -> fixed
- joint Joint6: origin xyz=0.34214 -0.028375 -0.41803 rpy=0 0 3.1416 -> xyz=-0.24 0 -0.272 rpy=0 -1.57 3.1416
- joint Joint7: axis 1 0 0 -> 0 0 1; origin xyz=0.044276 -0.018375 -0.014756 rpy=0 0 0 -> xyz=.03 0 -0.119 rpy=0 1.57 3.14
- joint ceiling_joint: origin xyz=0 0 -.37 rpy=0 0 0 -> xyz=0 0 0 rpy=0 0 0
