Commit message: Update URDF to include apriltags

File: ros2_ws/src/surg_bot/surg_bot_description/urdf/surg_bot.xacro (robot description, xacro)
@@ -144,4 +144,26 @@
   </collision>
 </link>
+<link name="base_connector_1">
+  <inertial>
+    <origin xyz="0.00473135651687414 -0.009256009227830791 0.014785071555408117" rpy="0 0 0"/>
+    <mass value="0.8564401248126177"/>
+    <inertia ixx="0.000724" iyy="0.00128" izz="0.00172" ixy="-1e-06" iyz="-0.0" ixz="-7.5e-05"/>
+  </inertial>
+  <visual>
+    <origin xyz="0.0 -0.0094 0.007" rpy="0 0 0"/>
+    <geometry>
+      <mesh filename="file://$(find surg_bot_description)/meshes/base_connector_1.stl" scale="0.001 0.001 0.001"/>
+    </geometry>
+    <material name="silver"/>
+  </visual>
+  <collision>
+    <origin xyz="0.0 -0.0094 0.007" rpy="0 0 0"/>
+    <geometry>
+      <mesh filename="file://$(find surg_bot_description)/meshes/base_connector_1.stl" scale="0.001 0.001 0.001"/>
+    </geometry>
+  </collision>
+</link>
+<link name="AprilTag0_1"/>
+<link name="AprilTag1_1"/>
 <joint name="joint0" type="revolute">
   <origin xyz="-1e-05 1e-05 -0.063784" rpy="0 0 0"/>
@@ -186,3 +208,18 @@
   <limit upper="3.141593" lower="-3.141593" effort="100" velocity="100"/>
 </joint>
+<joint name="rigid1" type="fixed">
+  <origin xyz="0.0 0.0094 -0.007" rpy="0 0 0"/>
+  <parent link="base_link"/>
+  <child link="base_connector_1"/>
+</joint>
+<joint name="tag0" type="fixed">
+  <origin xyz="-0.0572 -0.041877 0.0275" rpy="1.5708 0 0"/>
+  <parent link="base_connector_1"/>
+  <child link="AprilTag0_1"/>
+</joint>
+<joint name="tag1" type="fixed">
+  <origin xyz="-0.0572 0.023523 0.0275" rpy="-1.5708 -3.1416 0"/>
+  <parent link="base_connector_1"/>
+  <child link="AprilTag1_1"/>
+</joint>
 </robot>

Commit message: Got the offset working with the IK

File: ros2_ws/src/surg_bot/surg_bot_description/urdf/surg_bot.xacro (robot description, xacro)
@@ -46,5 +46,5 @@
 <link name="link2_1_1">
   <inertial>
-    <origin xyz="0.00022227782028544363 2.474064107253927e-05 -0.1173741177356839" rpy="0 0 0"/>
+    <origin xyz="0.000222277820202621 2.4740641813817415e-05 -0.11737411773568346" rpy="0 0 0"/>
     <mass value="3.3490679501648595"/>
     <inertia ixx="0.014417" iyy="0.014057" izz="0.002264" ixy="-1e-06" iyz="8e-06" ixz="-5.7e-05"/>
@@ -66,5 +66,5 @@
 <link name="link3_1">
   <inertial>
-    <origin xyz="0.13545922670739144 0.030192910577609006 0.00044866468088849976" rpy="0 0 0"/>
+    <origin xyz="0.1354592267935596 0.030192910648437193 0.00044866468104021173" rpy="0 0 0"/>
     <mass value="1.7602626049739658"/>
     <inertia ixx="0.001766" iyy="0.008244" izz="0.009744" ixy="2.4e-05" iyz="0.0" ixz="-2.6e-05"/>
@@ -86,5 +86,5 @@
 <link name="link4_1">
   <inertial>
-    <origin xyz="0.02605773282976529 -0.04507242712799745 8.675535075214347e-05" rpy="0 0 0"/>
+    <origin xyz="0.026057732789940877 -0.04507242698022944 8.680052417670003e-05" rpy="0 0 0"/>
     <mass value="1.4039319321687402"/>
     <inertia ixx="0.001418" iyy="0.001888" izz="0.002652" ixy="0.000674" iyz="2e-06" ixz="-4e-06"/>
@@ -104,9 +104,89 @@
   </collision>
 </link>
+<link name="fake_link_1">
+  <inertial>
+    <origin xyz="-0.0025000443408709893 8.946959404469842e-06 -8.268459717741816e-06" rpy="0 0 0"/>
+    <mass value="0.001098697673021953"/>
+    <inertia ixx="0.0" iyy="0.0" izz="0.0" ixy="-0.0" iyz="-0.0" ixz="0.0"/>
+  </inertial>
+  <visual>
+    <origin xyz="-0.014679 0.00143 0.302173" rpy="0 0 0"/>
+    <geometry>
+      <mesh filename="file://$(find surg_bot_description)/meshes/fake_link_1.stl" scale="0.001 0.001 0.001"/>
+    </geometry>
+    <material name="silver"/>
+  </visual>
+  <collision>
+    <origin xyz="-0.014679 0.00143 0.302173" rpy="0 0 0"/>
+    <geometry>
+      <mesh filename="file://$(find surg_bot_description)/meshes/fake_link_1.stl" scale="0.001 0.001 0.001"/>
+    </geometry>
+  </collision>
+</link>
+<link name="AprilTag0_1">
+  <inertial>
+    <origin xyz="-0.06120100000000133 -0.08805614874251824 0.05697699999999984" rpy="0 0 0"/>
+    <mass value="0.0628381454838991"/>
+    <inertia ixx="1.4e-05" iyy="2.9e-05" izz="1.4e-05" ixy="-0.0" iyz="0.0" ixz="-0.0"/>
+  </inertial>
+  <visual>
+    <origin xyz="-0.003901 -0.0572 0.036477" rpy="0 0 0"/>
+    <geometry>
+      <mesh filename="file://$(find surg_bot_description)/meshes/AprilTag0_1.stl" scale="0.001 0.001 0.001"/>
+    </geometry>
+    <material name="silver"/>
+  </visual>
+  <collision>
+    <origin xyz="-0.003901 -0.0572 0.036477" rpy="0 0 0"/>
+    <geometry>
+      <mesh filename="file://$(find surg_bot_description)/meshes/AprilTag0_1.stl" scale="0.001 0.001 0.001"/>
+    </geometry>
+  </collision>
+</link>
+<link name="base_connector_1">
+  <inertial>
+    <origin xyz="0.008739591761476772 -0.009261123091376765 0.013879262591046193" rpy="0 0 0"/>
+    <mass value="0.8045670076781538"/>
+    <inertia ixx="0.000675" iyy="0.001052" izz="0.001469" ixy="-1e-06" iyz="-0.0" ixz="-0.000124"/>
+  </inertial>
+  <visual>
+    <origin xyz="0.0 -0.0094 0.007" rpy="0 0 0"/>
+    <geometry>
+      <mesh filename="file://$(find surg_bot_description)/meshes/base_connector_1.stl" scale="0.001 0.001 0.001"/>
+    </geometry>
+    <material name="silver"/>
+  </visual>
+  <collision>
+    <origin xyz="0.0 -0.0094 0.007" rpy="0 0 0"/>
+    <geometry>
+      <mesh filename="file://$(find surg_bot_description)/meshes/base_connector_1.stl" scale="0.001 0.001 0.001"/>
+    </geometry>
+  </collision>
+</link>
+<link name="AprilTag1_1">
+  <inertial>
+    <origin xyz="-0.06120100000000168 -0.02589723471612928 -0.0024230000000001577" rpy="0 0 0"/>
+    <mass value="0.0628381454838991"/>
+    <inertia ixx="1.4e-05" iyy="2.9e-05" izz="1.4e-05" ixy="-0.0" iyz="0.0" ixz="0.0"/>
+  </inertial>
+  <visual>
+    <origin xyz="-0.003901 -0.0572 -0.022923" rpy="0 0 0"/>
+    <geometry>
+      <mesh filename="file://$(find surg_bot_description)/meshes/AprilTag1_1.stl" scale="0.001 0.001 0.001"/>
+    </geometry>
+    <material name="silver"/>
+  </visual>
+  <collision>
+    <origin xyz="-0.003901 -0.0572 -0.022923" rpy="0 0 0"/>
+    <geometry>
+      <mesh filename="file://$(find surg_bot_description)/meshes/AprilTag1_1.stl" scale="0.001 0.001 0.001"/>
+    </geometry>
+  </collision>
+</link>
 <link name="link5_1_1">
   <inertial>
-    <origin xyz="0.0001801099222721872 0.03886369124244137 0.0005895595584266555" rpy="0 0 0"/>
+    <origin xyz="-0.00044160365250938067 0.03911603505931648 3.168698741190523e-05" rpy="0 0 0"/>
     <mass value="0.38469776659589416"/>
-    <inertia ixx="0.000309" iyy="0.000348" izz="0.00055" ixy="0.0" iyz="-1e-06" ixz="0.0"/>
+    <inertia ixx="0.00055" iyy="0.000348" izz="0.000309" ixy="-0.0" iyz="-0.0" ixz="1e-06"/>
   </inertial>
   <visual>
@@ -124,46 +204,24 @@
   </collision>
 </link>
-<link name="end_effector_1_1">
-  <inertial>
-    <origin xyz="4.038171408361996e-07 9.114467316127806e-08 0.0025003140135481106" rpy="0 0 0"/>
-    <mass value="0.001098697673021953"/>
-    <inertia ixx="0.0" iyy="0.0" izz="0.0" ixy="0.0" iyz="-0.0" ixz="-0.0"/>
-  </inertial>
-  <visual>
-    <origin xyz="7.2e-05 0.001625 0.316972" rpy="0 0 0"/>
-    <geometry>
-      <mesh filename="file://$(find surg_bot_description)/meshes/end_effector_1_1.stl" scale="0.001 0.001 0.001"/>
-    </geometry>
-    <material name="silver"/>
-  </visual>
-  <collision>
-    <origin xyz="7.2e-05 0.001625 0.316972" rpy="0 0 0"/>
-    <geometry>
-      <mesh filename="file://$(find surg_bot_description)/meshes/end_effector_1_1.stl" scale="0.001 0.001 0.001"/>
-    </geometry>
-  </collision>
-</link>
-<link name="base_connector_1">
-  <inertial>
-    <origin xyz="0.00473135651687414 -0.009256009227830791 0.014785071555408117" rpy="0 0 0"/>
-    <mass value="0.8564401248126177"/>
-    <inertia ixx="0.000724" iyy="0.00128" izz="0.00172" ixy="-1e-06" iyz="-0.0" ixz="-7.5e-05"/>
-  </inertial>
-  <visual>
-    <origin xyz="0.0 -0.0094 0.007" rpy="0 0 0"/>
-    <geometry>
-      <mesh filename="file://$(find surg_bot_description)/meshes/base_connector_1.stl" scale="0.001 0.001 0.001"/>
-    </geometry>
-    <material name="silver"/>
-  </visual>
-  <collision>
-    <origin xyz="0.0 -0.0094 0.007" rpy="0 0 0"/>
-    <geometry>
-      <mesh filename="file://$(find surg_bot_description)/meshes/base_connector_1.stl" scale="0.001 0.001 0.001"/>
-    </geometry>
-  </collision>
-</link>
-<link name="AprilTag0_1"/>
-<link name="AprilTag1_1"/>
+<link name="end_effector_1">
+  <inertial>
+    <origin xyz="0.0009999117915723155 -4.233375403692912e-06 3.279256363175609e-06" rpy="0 0 0"/>
+    <mass value="0.05209742367356123"/>
+    <inertia ixx="2.8e-05" iyy="1.4e-05" izz="1.4e-05" ixy="-0.0" iyz="-0.0" ixz="0.0"/>
+  </inertial>
+  <visual>
+    <origin xyz="-0.014679 0.00143 0.302173" rpy="0 0 0"/>
+    <geometry>
+      <mesh filename="file://$(find surg_bot_description)/meshes/end_effector_1.stl" scale="0.001 0.001 0.001"/>
+    </geometry>
+    <material name="silver"/>
+  </visual>
+  <collision>
+    <origin xyz="-0.014679 0.00143 0.302173" rpy="0 0 0"/>
+    <geometry>
+      <mesh filename="file://$(find surg_bot_description)/meshes/end_effector_1.stl" scale="0.001 0.001 0.001"/>
+    </geometry>
+  </collision>
+</link>
 <joint name="joint0" type="revolute">
   <origin xyz="-1e-05 1e-05 -0.063784" rpy="0 0 0"/>
@@ -194,32 +252,39 @@
   <limit upper="2.268928" lower="-2.268928" effort="100" velocity="100"/>
 </joint>
+<joint name="joint5" type="revolute">
+  <origin xyz="0.014907 0.041545 4.9e-05" rpy="0 0 0"/>
+  <parent link="link5_1_1"/>
+  <child link="fake_link_1"/>
+  <axis xyz="0.999987 -0.003766 0.003299"/>
+  <limit upper="3.141593" lower="-3.141593" effort="100" velocity="100"/>
+</joint>
+<joint name="tag0" type="fixed">
+  <origin xyz="0.003901 0.0478 -0.029477" rpy="0 0 0"/>
+  <parent link="base_connector_1"/>
+  <child link="AprilTag0_1"/>
+</joint>
+<joint name="rigid1" type="fixed">
+  <origin xyz="0.0 0.0094 -0.007" rpy="0 0 0"/>
+  <parent link="base_link"/>
+  <child link="base_connector_1"/>
+</joint>
+<joint name="tag1" type="fixed">
+  <origin xyz="0.003901 0.0478 0.029923" rpy="0 0 0"/>
+  <parent link="base_connector_1"/>
+  <child link="AprilTag1_1"/>
+</joint>
 <joint name="joint4" type="revolute">
   <origin xyz="0.065091 -0.042116 0.000216" rpy="0 0 0"/>
   <parent link="link4_1"/>
   <child link="link5_1_1"/>
-  <axis xyz="0.003766 0.999993 1e-06"/>
+  <axis xyz="0.003766 0.999993 -0.0"/>
   <limit upper="2.268928" lower="-2.268928" effort="100" velocity="100"/>
 </joint>
-<joint name="joint5" type="revolute">
-  <origin xyz="0.000156 0.04135 -0.01475" rpy="0 0 0"/>
-  <parent link="link5_1_1"/>
-  <child link="end_effector_1_1"/>
-  <axis xyz="1.9e-05 1e-06 -1.0"/>
-  <limit upper="3.141593" lower="-3.141593" effort="100" velocity="100"/>
-</joint>
-<joint name="rigid1" type="fixed">
-  <origin xyz="0.0 0.0094 -0.007" rpy="0 0 0"/>
-  <parent link="base_link"/>
-  <child link="base_connector_1"/>
-</joint>
-<joint name="tag0" type="fixed">
-  <origin xyz="-0.0572 -0.041877 0.0275" rpy="1.5708 0 0"/>
-  <parent link="base_connector_1"/>
-  <child link="AprilTag0_1"/>
-</joint>
-<joint name="tag1" type="fixed">
-  <origin xyz="-0.0572 0.023523 0.0275" rpy="-1.5708 -3.1416 0"/>
-  <parent link="base_connector_1"/>
-  <child link="AprilTag1_1"/>
+<joint name="slider" type="prismatic">
+  <origin xyz="0.0 0.0 0.0" rpy="0 0 0"/>
+  <parent link="fake_link_1"/>
+  <child link="end_effector_1"/>
+  <axis xyz="0.999987 -0.003766 0.003299"/>
+  <limit upper="3.0" lower="0.0" effort="100" velocity="100"/>
 </joint>
 </robot>

File: ros2_ws/src/surg_bot/surg_bot_moveit_config/config/surg_bot.ros2_control.xacro (robot description, xacro)
@@ -44,4 +44,10 @@
                 </state_interface>
             </joint>
+            <joint name="slider">
+                <command_interface name="position"/>
+                <state_interface name="position">
+                  <param name="initial_value">${initial_positions['slider']}</param>
+                </state_interface>
+            </joint>
         </ros2_control>
     </xacro:macro>

Commit message: Fix coordinates of April Tags on URDF

File: ros2_ws/src/surg_bot/surg_bot_description/urdf/surg_bot.xacro (robot description, xacro)
@@ -124,24 +124,5 @@
   </collision>
 </link>
-<link name="AprilTag0_1">
-  <inertial>
-    <origin xyz="-0.06120100000000133 -0.08805614874251824 0.05697699999999984" rpy="0 0 0"/>
-    <mass value="0.0628381454838991"/>
-    <inertia ixx="1.4e-05" iyy="2.9e-05" izz="1.4e-05" ixy="-0.0" iyz="0.0" ixz="-0.0"/>
-  </inertial>
-  <visual>
-    <origin xyz="-0.003901 -0.0572 0.036477" rpy="0 0 0"/>
-    <geometry>
-      <mesh filename="file://$(find surg_bot_description)/meshes/AprilTag0_1.stl" scale="0.001 0.001 0.001"/>
-    </geometry>
-    <material name="silver"/>
-  </visual>
-  <collision>
-    <origin xyz="-0.003901 -0.0572 0.036477" rpy="0 0 0"/>
-    <geometry>
-      <mesh filename="file://$(find surg_bot_description)/meshes/AprilTag0_1.stl" scale="0.001 0.001 0.001"/>
-    </geometry>
-  </collision>
-</link>
+<link name="AprilTag0_1"/>
 <link name="base_connector_1">
   <inertial>
@@ -164,24 +145,5 @@
   </collision>
 </link>
-<link name="AprilTag1_1">
-  <inertial>
-    <origin xyz="-0.06120100000000168 -0.02589723471612928 -0.0024230000000001577" rpy="0 0 0"/>
-    <mass value="0.0628381454838991"/>
-    <inertia ixx="1.4e-05" iyy="2.9e-05" izz="1.4e-05" ixy="-0.0" iyz="0.0" ixz="0.0"/>
-  </inertial>
-  <visual>
-    <origin xyz="-0.003901 -0.0572 -0.022923" rpy="0 0 0"/>
-    <geometry>
-      <mesh filename="file://$(find surg_bot_description)/meshes/AprilTag1_1.stl" scale="0.001 0.001 0.001"/>
-    </geometry>
-    <material name="silver"/>
-  </visual>
-  <collision>
-    <origin xyz="-0.003901 -0.0572 -0.022923" rpy="0 0 0"/>
-    <geometry>
-      <mesh filename="file://$(find surg_bot_description)/meshes/AprilTag1_1.stl" scale="0.001 0.001 0.001"/>
-    </geometry>
-  </collision>
-</link>
+<link name="AprilTag1_1"/>
 <link name="link5_1_1">
   <inertial>
@@ -259,9 +221,4 @@
   <limit upper="3.141593" lower="-3.141593" effort="100" velocity="100"/>
 </joint>
-<joint name="tag0" type="fixed">
-  <origin xyz="0.003901 0.0478 -0.029477" rpy="0 0 0"/>
-  <parent link="base_connector_1"/>
-  <child link="AprilTag0_1"/>
-</joint>
 <joint name="rigid1" type="fixed">
   <origin xyz="0.0 0.0094 -0.007" rpy="0 0 0"/>
@@ -269,6 +226,11 @@
   <child link="base_connector_1"/>
 </joint>
+<joint name="tag0" type="fixed">
+  <origin xyz="-0.0572 -0.041877 0.0275" rpy="1.5708 0 0"/>
+  <parent link="base_connector_1"/>
+  <child link="AprilTag0_1"/>
+</joint>
 <joint name="tag1" type="fixed">
-  <origin xyz="0.003901 0.0478 0.029923" rpy="0 0 0"/>
+  <origin xyz="-0.0572 0.023523 0.0275" rpy="-1.5708 -3.1416 0"/>
   <parent link="base_connector_1"/>
   <child link="AprilTag1_1"/>
