File: Electrical/schematic/schematic.kicad_sch (KiCad schematic)
At the start: 18 parts, among them M1 Joint 0 Stepper, M2 Joint 1 Stepper

Commit message: Rev 1 of electrical schematic
Connections:
- new net: U10. (12), U13. (VCC) (x4)
Other:
- note added: "MCU-1"
- note added: "MCU-2"
Changed lines of the file:
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@@
+		)
+	)
+	(text "MCU-2"
+		(exclude_from_sim no)
+		(at 93.472 57.658 0)
+		(effects
+			(font
+				(size 1.27 1.27)
+			)
 		)
 	)
@@
 				(thickness 0.254)
 				(bold yes)
+			)
+		)
+	)
+	(text "MCU-1"
+		(exclude_from_sim no)
+		(at 248.412 93.472 0)
+		(effects
+			(font
+				(size 1.27 1.27)
 			)
 		)
@@
 	(wire
 		(pts
-			(xy 128.27 123.19) (xy 147.32 123.19)
-		)
-		(stroke
-			(width 0)
-			(type default)
-		)
-	)
-	(wire
-		(pts
 			(xy 203.2 138.43) (xy 208.28 138.43)
 		)
@@
 	(wire
 		(pts
-			(xy 128.27 138.43) (xy 147.32 138.43)
-		)
-		(stroke
-			(width 0)
-			(type default)
-		)
-	)
-	(wire
-		(pts
 			(xy 91.44 78.74) (xy 110.49 78.74)
 		)
@@
 	(wire
 		(pts
-			(xy 128.27 120.65) (xy 147.32 120.65)
+			(xy 33.02 138.43) (xy 35.56 138.43)
 		)
 		(stroke
@@
 	(wire
 		(pts
-			(xy 128.27 125.73) (xy 147.32 125.73)
-		)
-		(stroke
-			(width 0)
-			(type default)
-		)
-	)
-	(wire
-		(pts
 			(xy 246.38 127) (xy 255.27 127)
 		)
@@
 	(wire
 		(pts
-			(xy 128.27 130.81) (xy 147.32 130.81)
-		)
-		(stroke
-			(width 0)
-			(type default)
-		)
-	)
-	(wire
-		(pts
 			(xy 166.37 140.97) (xy 184.15 140.97)
 		)
@@
 	(wire
 		(pts
-			(xy 128.27 146.05) (xy 147.32 146.05)
-		)
-		(stroke
-			(width 0)
-			(type default)
-		)
-	)
-	(wire
-		(pts
 			(xy 81.28 49.53) (xy 93.98 49.53)
 		)
@@
 	(wire
 		(pts
-			(xy 128.27 135.89) (xy 147.32 135.89)
-		)
-		(stroke
-			(width 0)
-			(type default)
-		)
-	)
-	(wire
-		(pts
 			(xy 54.61 31.75) (xy 54.61 66.04)
 		)
@@
 	(wire
 		(pts
-			(xy 128.27 133.35) (xy 147.32 133.35)
-		)
-		(stroke
-			(width 0)
-			(type default)
-		)
-	)
-	(wire
-		(pts
 			(xy 172.72 92.71) (xy 161.29 92.71)
 		)
@@
 	(wire
 		(pts
-			(xy 128.27 128.27) (xy 147.32 128.27)
-		)
-		(stroke
-			(width 0)
-			(type default)
-		)
-	)
-	(wire
-		(pts
 			(xy 97.79 130.81) (xy 115.57 130.81)
 		)
@@
 	(wire
 		(pts
-			(xy 128.27 143.51) (xy 147.32 143.51)
-		)
-		(stroke
-			(width 0)
-			(type default)
-		)
-	)
-	(wire
-		(pts
 			(xy 246.38 124.46) (xy 255.27 124.46)
 		)
@@
 	(wire
 		(pts
-			(xy 128.27 140.97) (xy 147.32 140.97)
-		)
-		(stroke
-			(width 0)
-			(type default)
-		)
-	)
-	(wire
-		(pts
 			(xy 48.26 71.12) (xy 66.04 71.12)
 		)
@@
 	(wire
 		(pts
-			(xy 128.27 148.59) (xy 147.32 148.59)
-		)
-		(stroke
-			(width 0)
-			(type default)
-		)
-	)
-	(wire
-		(pts
 			(xy 203.2 140.97) (xy 210.82 140.97)
 		)
@@
 		)
 		(stroke
-			(width 0)
-			(type default)
-		)
-	)
-	(wire
-		(pts
-			(xy 24.13 138.43) (xy 35.56 138.43)
-		)
-		(stroke
