File: Electrical/Surgery_Lamp_Control_Board/KiCad/Surgery_Lamp_Control_PCB.kicad_sch (KiCad schematic)
At the start: 21 parts, among them J1 OSTVN05A150, J2 Headlamp, J3 Joint 1 Encoder, J4 Joint 2 Encoder, Q1 BSS138, Q2 BSS138

Commit message: Update platform configuration for mcu2 and clean up KiCad files; remove unused autosave and lock files
Parts:
- added A2: Pololu_Breakout_DRV8825, Module:Pololu_Breakout-16_15.2x20.3mm, symbol Driver_Motor:Pololu_Breakout_DRV8825
- added C6: 10uF, Capacitor_SMD:C_0805_2012Metric, symbol Device:C
- added C7: 0.1uF, Capacitor_SMD:C_0805_2012Metric, symbol Device:C
- added C8: 47uF, Alec_lib:CAP_6.3 X 5.8_PAN, symbol Device:C_Polarized
- added J10: joint2, Connector_PinSocket_2.54mm:PinSocket_1x03_P2.54mm_Vertical, symbol Connector_Generic:Conn_01x03
- added J11: joint3, Connector_PinSocket_2.54mm:PinSocket_1x04_P2.54mm_Vertical, symbol Connector_Generic:Conn_01x04
- added J12: joint4, Connector_PinSocket_2.54mm:PinSocket_1x04_P2.54mm_Vertical, symbol Connector_Generic:Conn_01x04
- added J9: Stepper, Connector_PinSocket_2.54mm:PinSocket_1x04_P2.54mm_Vertical, symbol Connector_Generic:Conn_01x04
- added Q10, Q7, Q8, Q9: BSS138, Package_TO_SOT_SMD:SOT-23-3, symbol Transistor_FET:BSS138
- added R18, R19, R20, R21, R25, R26: 10k, Resistor_SMD:R_0805_2012Metric, symbol Device:R_US
- added R22: 120, Resistor_SMD:R_0805_2012Metric, symbol Device:R_US
- added R23, R24: 20k, Resistor_SMD:R_0805_2012Metric, symbol Device:R_US
- added U3: MAX485E, Package_SO:SOIC-8-1EP_3.9x4.9mm_P1.27mm_EP2.29x3mm, symbol Interface_UART:MAX485E
- added U4: PCA9685PW, Package_SO:TSSOP-28_4.4x9.7mm_P0.65mm, symbol Alecs_Lib:PCA9685PW
Connections:
- net 24V: now also A2.8 (VMOT), C8.1, J10.2 (Pin_2)
- net 3V3: now also A2.10 (M0), A2.11 (M1), A2.12 (M2), A2.13 (~{RST}), A2.14 (~{SLP}), Q10.1 (G), Q7.1 (G), Q8.1 (G), Q9.1 (G), R18.1, R19.1
- net 5V: now also C6.1, C7.1, J11.3 (Pin_3), J12.3 (Pin_3), R20.1, R21.1, R23.1, R25.1, R26.1, U3.8 (VCC), U4.28 (VDD)
- net DIR: now also A2.16 (DIR)
- net GND: now also A2.1 (GND), A2.7 (GND), C6.2, C7.2, C8.2, J10.3 (Pin_3), J11.4 (Pin_4), J12.4 (Pin_4), R24.2, U3.5 (GND), U3.9, U4.1 (A0), U4.14 (VSS), U4.2 (A1), U4.23 (*OE), U4.3 (A2), U4.4 (A3), U4.5 (A4)
- net RS+: now also R22.1, R23.2, U3.6 (A)
- net RS-: now also R22.2, R24.1, U3.7 (B)
- net RX: now also Q7.2 (S), R18.2
- net SCL1: now also Q10.2 (S)
- net SDA1: now also Q9.2 (S)
- net STEP: now also A2.15 (STEP)
- net TX: now also Q8.2 (S), R19.2
- net joint3_Feedback: now also J11.1 (Pin_1)
- net joint4_Feedback: now also J12.1 (Pin_1)
- net RS_Enable: now reaches MCU1.9 (GPIO6)
- net RS_Enable: now also U3.2 (~{RE}), U3.3 (DE)
- new net: Q8.3 (D), R21.2, U3.4 (DI)
- new net: J10.1 (Pin_1), U4.6 (LED0)
- new net: Q7.3 (D), R20.2, U3.1 (RO)
- new net: A2.3 (A2), J9.4 (Pin_4)
- new net: A2.4 (A1), J9.3 (Pin_3)
- new net: A2.5 (B1), J9.2 (Pin_2)
- new net: A2.6 (B2), J9.1 (Pin_1)
- new net: J12.2 (Pin_2), U4.8 (LED2)
- new net: J11.2 (Pin_2), U4.7 (LED1)
- new net SCL1_5V: Q10.3 (D), R26.2, U4.26 (SCL)
- new net SDA1_5V: Q9.3 (D), R25.2, U4.27 (SDA)
- no-connect marks 19 -> 35
Other:
- removed sheet A4988
- removed sheet MAX485
- removed sheet PCA9685
- note added: "Connectors"
- note added: "Logic Converters"
- note added: "MCU1"
- note added: "Servo Control"
- note added: "Stepper Control"
- note added: "TTL to RS-485"
- note added: "joint2"
- note added: "joint3"
- note added: "joint4"
- moved on the sheet: C1, C2, H1, H2, H3, H4, J1, J2, J3, J4, MCU1, Q1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
