Commit message: Remove lamp_1 mesh and update URDF references to link5_1 and end_effector_1

File: ros2_ws/src/surg_bot_description/urdf/surg_bot.xacro (robot description, xacro)
@@ -104,5 +104,5 @@
   </collision>
 </link>
-<link name="lamp_1">
+<link name="link5_1">
   <inertial>
     <origin xyz="-3.290383739201763e-05 -0.04081342288708706 0.000588083950290641" rpy="0 0 0"/>
@@ -113,5 +113,5 @@
     <origin xyz="0.156734 -0.045503 0.232013" rpy="0 0 0"/>
     <geometry>
-      <mesh filename="file://$(find surg_bot_description)/meshes/lamp_1.stl" scale="0.001 0.001 0.001"/>
+      <mesh filename="file://$(find surg_bot_description)/meshes/link5_1.stl" scale="0.001 0.001 0.001"/>
     </geometry>
     <material name="silver"/>
@@ -120,5 +120,25 @@
     <origin xyz="0.156734 -0.045503 0.232013" rpy="0 0 0"/>
     <geometry>
-      <mesh filename="file://$(find surg_bot_description)/meshes/lamp_1.stl" scale="0.001 0.001 0.001"/>
+      <mesh filename="file://$(find surg_bot_description)/meshes/link5_1.stl" scale="0.001 0.001 0.001"/>
+    </geometry>
+  </collision>
+</link>
+<link name="end_effector_1">
+  <inertial>
+    <origin xyz="-4.215304917343232e-07 1.064626750394912e-07 0.0025002918773591454" rpy="0 0 0"/>
+    <mass value="0.0010986976730219535"/>
+    <inertia ixx="0.0" iyy="0.0" izz="0.0" ixy="-0.0" iyz="0.0" ixz="-0.0"/>
+  </inertial>
+  <visual>
+    <origin xyz="0.156733 -0.002103 0.246763" rpy="0 0 0"/>
+    <geometry>
+      <mesh filename="file://$(find surg_bot_description)/meshes/end_effector_1.stl" scale="0.001 0.001 0.001"/>
+    </geometry>
+    <material name="silver"/>
+  </visual>
+  <collision>
+    <origin xyz="0.156733 -0.002103 0.246763" rpy="0 0 0"/>
+    <geometry>
+      <mesh filename="file://$(find surg_bot_description)/meshes/end_effector_1.stl" scale="0.001 0.001 0.001"/>
     </geometry>
   </collision>
@@ -153,7 +173,12 @@
   <origin xyz="-0.06905 0.05035 -1e-06" rpy="0 0 0"/>
   <parent link="link4_1"/>
-  <child link="lamp_1"/>
+  <child link="link5_1"/>
   <axis xyz="-0.0 -1.0 0.0"/>
   <limit upper="2.268928" lower="-2.268928" effort="100" velocity="100"/>
 </joint>
+<joint name="Rigid 6" type="fixed">
+  <origin xyz="1e-06 -0.0434 -0.01475" rpy="0 0 0"/>
+  <parent link="link5_1"/>
+  <child link="end_effector_1"/>
+</joint>
 </robot>

Commit message: Remove obsolete mesh files and update URDF references for improved model accuracy

File: ros2_ws/src/surg_bot_description/urdf/surg_bot.xacro (robot description, xacro)
@@ -6,6 +6,6 @@
 <link name="base_link">
   <inertial>
-    <origin xyz="-0.006200037417416256 -0.004904380492643843 0.04172142536428126" rpy="0 0 0"/>
-    <mass value="0.40694896195118685"/>
+    <origin xyz="-0.06278565204512523 -0.018517571033498794 0.006090755429043733" rpy="0 0 0"/>
+    <mass value="0.406948961951185"/>
     <inertia ixx="0.000314" iyy="0.000315" izz="0.000167" ixy="-0.0" iyz="0.0" ixz="0.0"/>
   </inertial>
@@ -24,161 +24,161 @@
   </collision>
 </link>
-<link name="link1_1">
+<link name="link1_1_1">
   <inertial>
-    <origin xyz="0.1600002369578537 5.540348034358336e-06 -0.017608332454859398" rpy="0 0 0"/>
-    <mass value="8.367890341080882"/>
-    <inertia ixx="0.012225" iyy="0.118361" izz="0.124365" ixy="-0.0" iyz="-0.0" ixz="-0.001924"/>
+    <origin xyz="-0.16001041625629978 -1.5556549154669558e-05 -0.017608002390173735" rpy="0 0 0"/>
+    <mass value="8.367890341080868"/>
+    <inertia ixx="0.012225" iyy="0.118361" izz="0.124365" ixy="-0.0" iyz="-0.0" ixz="0.001924"/>
   </inertial>
   <visual>
-    <origin xyz="0.00617 0.004897 -0.007492" rpy="0 0 0"/>
+    <origin xyz="0.062755 0.01851 0.028139" rpy="0 0 0"/>
     <geometry>
-      <mesh filename="file://$(find surg_bot_description)/meshes/link1_1.stl" scale="0.001 0.001 0.001"/>
+      <mesh filename="file://$(find surg_bot_description)/meshes/link1_1_1.stl" scale="0.001 0.001 0.001"/>
     </geometry>
     <material name="silver"/>
   </visual>
   <collision>
-    <origin xyz="0.00617 0.004897 -0.007492" rpy="0 0 0"/>
+    <origin xyz="0.062755 0.01851 0.028139" rpy="0 0 0"/>
     <geometry>
-      <mesh filename="file://$(find surg_bot_description)/meshes/link1_1.stl" scale="0.001 0.001 0.001"/>
+      <mesh filename="file://$(find surg_bot_description)/meshes/link1_1_1.stl" scale="0.001 0.001 0.001"/>
     </geometry>
   </collision>
 </link>
-<link name="link2_1">
+<link name="link2_1_1">
   <inertial>
-    <origin xyz="-0.0002220234333368265 -2.5471499862192437e-05 -0.11737370019061386" rpy="0 0 0"/>
-    <mass value="3.3490679501648546"/>
-    <inertia ixx="0.014417" iyy="0.014057" izz="0.002264" ixy="0.0" iyz="-8e-06" ixz="5.7e-05"/>
+    <origin xyz="0.0002218441341833577 2.54552988030593e-05 -0.11737437012585125" rpy="0 0 0"/>
+    <mass value="3.3490679501648395"/>
+    <inertia ixx="0.014417" iyy="0.014057" izz="0.002264" ixy="0.0" iyz="8e-06" ixz="-5.7e-05"/>
   </inertial>
   <visual>
-    <origin xyz="-0.31384 0.004907 0.027725" rpy="0 0 0"/>
+    <origin xyz="0.382775 0.01851 0.063355" rpy="0 0 0"/>
     <geometry>
-      <mesh filename="file://$(find surg_bot_description)/meshes/link2_1.stl" scale="0.001 0.001 0.001"/>
+      <mesh filename="file://$(find surg_bot_description)/meshes/link2_1_1.stl" scale="0.001 0.001 0.001"/>
     </geometry>
     <material name="silver"/>
   </visual>
   <collision>
-    <origin xyz="-0.31384 0.004907 0.027725" rpy="0 0 0"/>
+    <origin xyz="0.382775 0.01851 0.063355" rpy="0 0 0"/>
     <geometry>
-      <mesh filename="file://$(find surg_bot_description)/meshes/link2_1.stl" scale="0.001 0.001 0.001"/>
+      <mesh filename="file://$(find surg_bot_description)/meshes/link2_1_1.stl" scale="0.001 0.001 0.001"/>
     </geometry>
   </collision>
 </link>
-<link name="link3_1">
+<link name="link3_1_1">
   <inertial>
-    <origin xyz="-0.2110414657474451 0.030754237211609886 -2.12340437225067e-06" rpy="0 0 0"/>
-    <mass value="4.3450582468708445"/>
-    <inertia ixx="0.003399" iyy="0.040399" izz="0.043145" ixy="4.2e-05" iyz="0.0" ixz="-0.0"/>
+    <origin xyz="0.21104127231910477 0.030645747745601536 -1.8019677435199277e-06" rpy="0 0 0"/>
+    <mass value="4.345058247420326"/>
+    <inertia ixx="0.003399" iyy="0.040399" izz="0.043145" ixy="4.2e-05" iyz="-0.0" ixz="0.0"/>
   </inertial>
   <visual>
-    <origin xyz="-0.31383 0.035697 0.232008" rpy="0 0 0"/>
+    <origin xyz="0.382765 0.04912 0.267639" rpy="0 0 0"/>
     <geometry>
-      <mesh filename="file://$(find surg_bot_description)/meshes/link3_1.stl" scale="0.001 0.001 0.001"/>
+      <mesh filename="file://$(find surg_bot_description)/meshes/link3_1_1.stl" scale="0.001 0.001 0.001"/>
     </geometry>
     <material name="silver"/>
   </visual>
   <collision>
-    <origin xyz="-0.31383 0.035697 0.232008" rpy="0 0 0"/>
+    <origin xyz="0.382765 0.04912 0.267639" rpy="0 0 0"/>
     <geometry>
-      <mesh filename="file://$(find surg_bot_description)/meshes/link3_1.stl" scale="0.001 0.001 0.001"/>
+      <mesh filename="file://$(find surg_bot_description)/meshes/link3_1_1.stl" scale="0.001 0.001 0.001"/>
     </geometry>
   </collision>
 </link>
-<link name="link4_1">
+<link name="link4_1_1">
   <inertial>
-    <origin xyz="-0.029750200264352225 0.049481837853942605 -2.927728003704333e-05" rpy="0 0 0"/>
-    <mass value="1.5005041494350506"/>
-    <inertia ixx="0.00166" iyy="0.002022" izz="0.002998" ixy="0.000773" iyz="0.0" ixz="-2e-06"/>
+    <origin xyz="0.029751892519794897 -0.049482100868121964 -2.921340474681955e-05" rpy="0 0 0"/>
+    <mass value="1.5005223483382892"/>
+    <inertia ixx="0.00166" iyy="0.002022" izz="0.002999" ixy="0.000773" iyz="-0.0" ixz="2e-06"/>
   </inertial>
   <visual>
-    <origin xyz="0.087684 0.004847 0.232012" rpy="0 0 0"/>
+    <origin xyz="-0.018748 0.01857 0.267643" rpy="0 0 0"/>
     <geometry>
-      <mesh filename="file://$(find surg_bot_description)/meshes/link4_1.stl" scale="0.001 0.001 0.001"/>
+      <mesh filename="file://$(find surg_bot_description)/meshes/link4_1_1.stl" scale="0.001 0.001 0.001"/>
     </geometry>
     <material name="silver"/>
   </visual>
   <collision>
-    <origin xyz="0.087684 0.004847 0.232012" rpy="0 0 0"/>
+    <origin xyz="-0.018748 0.01857 0.267643" rpy="0 0 0"/>
     <geometry>
-      <mesh filename="file://$(find surg_bot_description)/meshes/link4_1.stl" scale="0.001 0.001 0.001"/>
+      <mesh filename="file://$(find surg_bot_description)/meshes/link4_1_1.stl" scale="0.001 0.001 0.001"/>
     </geometry>
   </collision>
 </link>
-<link name="link5_1">
+<link name="link5_1_1">
   <inertial>
-    <origin xyz="-3.290383739201763e-05 -0.04081342288708706 0.000588083950290641" rpy="0 0 0"/>
-    <mass value="0.38564981413000793"/>
-    <inertia ixx="0.000311" iyy="0.000348" izz="0.000552" ixy="-0.0" iyz="1e-06" ixz="-0.0"/>
+    <origin xyz="3.372453495051331e-05 0.040813406687341375 0.000587414034003364" rpy="0 0 0"/>
+    <mass value="0.3856498141159764"/>
+    <inertia ixx="0.000311" iyy="0.000348" izz="0.000552" ixy="-0.0" iyz="-1e-06" ixz="0.0"/>
   </inertial>
   <visual>
-    <origin xyz="0.156734 -0.045503 0.232013" rpy="0 0 0"/>
+    <origin xyz="-0.087798 0.06892 0.267643" rpy="0 0 0"/>
     <geometry>
-      <mesh filename="file://$(find surg_bot_description)/meshes/link5_1.stl" scale="0.001 0.001 0.001"/>
+      <mesh filename="file://$(find surg_bot_description)/meshes/link5_1_1.stl" scale="0.001 0.001 0.001"/>
     </geometry>
     <material name="silver"/>
   </visual>
   <collision>
-    <origin xyz="0.156734 -0.045503 0.232013" rpy="0 0 0"/>
+    <origin xyz="-0.087798 0.06892 0.267643" rpy="0 0 0"/>
     <geometry>
-      <mesh filename="file://$(find surg_bot_description)/meshes/link5_1.stl" scale="0.001 0.001 0.001"/>
+      <mesh filename="file://$(find surg_bot_description)/meshes/link5_1_1.stl" scale="0.001 0.001 0.001"/>
     </geometry>
   </collision>
 </link>
-<link name="end_effector_1">
+<link name="end_effector_1_1">
   <inertial>
-    <origin xyz="-4.215304917343232e-07 1.064626750394912e-07 0.0025002918773591454" rpy="0 0 0"/>
-    <mass value="0.0010986976730219535"/>
-    <inertia ixx="0.0" iyy="0.0" izz="0.0" ixy="-0.0" iyz="0.0" ixz="-0.0"/>
+    <origin xyz="1.4572522974432012e-07 -1.2266364841223565e-07 -0.0025003780571151712" rpy="0 0 0"/>
+    <mass value="0.001098697673021953"/>
+    <inertia ixx="0.0" iyy="0.0" izz="0.0" ixy="0.0" iyz="0.0" ixz="0.0"/>
   </inertial>
   <visual>
-    <origin xyz="0.156733 -0.002103 0.246763" rpy="0 0 0"/>
+    <origin xyz="-0.087798 0.02552 0.282393" rpy="0 0 0"/>
     <geometry>
-      <mesh filename="file://$(find surg_bot_description)/meshes/end_effector_1.stl" scale="0.001 0.001 0.001"/>
+      <mesh filename="file://$(find surg_bot_description)/meshes/end_effector_1_1.stl" scale="0.001 0.001 0.001"/>
     </geometry>
     <material name="silver"/>
   </visual>
   <collision>
-    <origin xyz="0.156733 -0.002103 0.246763" rpy="0 0 0"/>
+    <origin xyz="-0.087798 0.02552 0.282393" rpy="0 0 0"/>
     <geometry>
-      <mesh filename="file://$(find surg_bot_description)/meshes/end_effector_1.stl" scale="0.001 0.001 0.001"/>
+      <mesh filename="file://$(find surg_bot_description)/meshes/end_effector_1_1.stl" scale="0.001 0.001 0.001"/>
     </geometry>
   </collision>
 </link>
-<joint name="Revolute 1" type="continuous">
-  <origin xyz="-0.00617 -0.004897 0.007492" rpy="0 0 0"/>
+<joint name="Revolute 7" type="continuous">
+  <origin xyz="-0.062755 -0.01851 -0.028139" rpy="0 0 0"/>
   <parent link="base_link"/>
-  <child link="link1_1"/>
+  <child link="link1_1_1"/>
+  <axis xyz="-0.0 0.0 1.0"/>
+</joint>
+<joint name="Revolute 8" type="continuous">
+  <origin xyz="-0.32002 0.0 -0.035216" rpy="0 0 0"/>
+  <parent link="link1_1_1"/>
+  <child link="link2_1_1"/>
   <axis xyz="0.0 0.0 1.0"/>
 </joint>
-<joint name="Revolute 2" type="continuous">
-  <origin xyz="0.32001 -1e-05 -0.035217" rpy="0 0 0"/>
-  <parent link="link1_1"/>
-  <child link="link2_1"/>
-  <axis xyz="-0.0 0.0 1.0"/>
+<joint name="Revolute 9" type="revolute">
+  <origin xyz="1e-05 -0.03061 -0.204284" rpy="0 0 0"/>
+  <parent link="link2_1_1"/>
+  <child link="link3_1_1"/>
+  <axis xyz="0.0 -1.0 0.0"/>
+  <limit upper="0.174533" lower="-1.570796" effort="100" velocity="100"/>
 </joint>
-<joint name="Revolute 3" type="revolute">
-  <origin xyz="-1e-05 -0.03079 -0.204283" rpy="0 0 0"/>
-  <parent link="link2_1"/>
-  <child link="link3_1"/>
-  <axis xyz="-0.0 -1.0 0.0"/>
-  <limit upper="1.570796" lower="-0.174533" effort="100" velocity="100"/>
-</joint>
-<joint name="Revolute 4" type="revolute">
-  <origin xyz="-0.401514 0.03085 -4e-06" rpy="0 0 0"/>
-  <parent link="link3_1"/>
-  <child link="link4_1"/>
-  <axis xyz="-1.0 0.0 -1e-05"/>
+<joint name="Revolute 10" type="revolute">
+  <origin xyz="0.401513 0.03055 -4e-06" rpy="0 0 0"/>
+  <parent link="link3_1_1"/>
+  <child link="link4_1_1"/>
+  <axis xyz="1.0 -0.0 -1e-05"/>
   <limit upper="2.268928" lower="-2.268928" effort="100" velocity="100"/>
 </joint>
-<joint name="Revolute 5" type="revolute">
-  <origin xyz="-0.06905 0.05035 -1e-06" rpy="0 0 0"/>
-  <parent link="link4_1"/>
-  <child link="link5_1"/>
-  <axis xyz="-0.0 -1.0 0.0"/>
+<joint name="Revolute 11" type="revolute">
+  <origin xyz="0.06905 -0.05035 0.0" rpy="0 0 0"/>
+  <parent link="link4_1_1"/>
+  <child link="link5_1_1"/>
+  <axis xyz="0.0 1.0 0.0"/>
   <limit upper="2.268928" lower="-2.268928" effort="100" velocity="100"/>
 </joint>
-<joint name="Rigid 6" type="fixed">
-  <origin xyz="1e-06 -0.0434 -0.01475" rpy="0 0 0"/>
-  <parent link="link5_1"/>
-  <child link="end_effector_1"/>
+<joint name="Rigid 12" type="fixed">
+  <origin xyz="0.0 0.0434 -0.01475" rpy="0 0 0"/>
+  <parent link="link5_1_1"/>
+  <child link="end_effector_1_1"/>
 </joint>
 </robot>

Commit message: Change description to fix base origin

File: ros2_ws/src/surg_bot_description/urdf/surg_bot.xacro (robot description, xacro)
@@ -6,6 +6,6 @@
 <link name="base_link">
   <inertial>
-    <origin xyz="-0.06278565204512523 -0.018517571033498794 0.006090755429043733" rpy="0 0 0"/>
-    <mass value="0.406948961951185"/>
+    <origin xyz="-4.031295976229773e-05 2.551630137478745e-06 -0.02955399218078996" rpy="0 0 0"/>
+    <mass value="0.4069489619511855"/>
     <inertia ixx="0.000314" iyy="0.000315" izz="0.000167" ixy="-0.0" iyz="0.0" ixz="0.0"/>
   </inertial>
@@ -26,10 +26,10 @@
 <link name="link1_1_1">
   <inertial>
-    <origin xyz="-0.16001041625629978 -1.5556549154669558e-05 -0.017608002390173735" rpy="0 0 0"/>
+    <origin xyz="-0.16001007717101118 -1.5433885539871676e-05 -0.01760775000004905" rpy="0 0 0"/>
     <mass value="8.367890341080868"/>
-    <inertia ixx="0.012225" iyy="0.118361" izz="0.124365" ixy="-0.0" iyz="-0.0" ixz="0.001924"/>
+    <inertia ixx="0.012225" iyy="0.118361" izz="0.124365" ixy="0.0" iyz="0.0" ixz="0.001924"/>
   </inertial>
   <visual>
-    <origin xyz="0.062755 0.01851 0.028139" rpy="0 0 0"/>
+    <origin xyz="1e-05 -1e-05 0.063784" rpy="0 0 0"/>
     <geometry>
       <mesh filename="file://$(find surg_bot_description)/meshes/link1_1_1.stl" scale="0.001 0.001 0.001"/>
@@ -38,5 +38,5 @@
   </visual>
   <collision>
-    <origin xyz="0.062755 0.01851 0.028139" rpy="0 0 0"/>
+    <origin xyz="1e-05 -1e-05 0.063784" rpy="0 0 0"/>
     <geometry>
       <mesh filename="file://$(find surg_bot_description)/meshes/link1_1_1.stl" scale="0.001 0.001 0.001"/>
@@ -46,10 +46,10 @@
 <link name="link2_1_1">
   <inertial>
-    <origin xyz="0.0002218441341833577 2.54552988030593e-05 -0.11737437012585125" rpy="0 0 0"/>
-    <mass value="3.3490679501648395"/>
+    <origin xyz="0.00022218321954753373 2.5577962440391797e-05 -0.11737411773568335" rpy="0 0 0"/>
+    <mass value="3.3490679501648595"/>
     <inertia ixx="0.014417" iyy="0.014057" izz="0.002264" ixy="0.0" iyz="8e-06" ixz="-5.7e-05"/>
   </inertial>
   <visual>
-    <origin xyz="0.382775 0.01851 0.063355" rpy="0 0 0"/>
+    <origin xyz="0.32003 -1e-05 0.099" rpy="0 0 0"/>
     <geometry>
       <mesh filename="file://$(find surg_bot_description)/meshes/link2_1_1.stl" scale="0.001 0.001 0.001"/>
@@ -58,5 +58,5 @@
   </visual>
   <collision>
-    <origin xyz="0.382775 0.01851 0.063355" rpy="0 0 0"/>
+    <origin xyz="0.32003 -1e-05 0.099" rpy="0 0 0"/>
     <geometry>
       <mesh filename="file://$(find surg_bot_description)/meshes/link2_1_1.stl" scale="0.001 0.001 0.001"/>
@@ -66,10 +66,10 @@
 <link name="link3_1_1">
   <inertial>
-    <origin xyz="0.21104127231910477 0.030645747745601536 -1.8019677435199277e-06" rpy="0 0 0"/>
-    <mass value="4.345058247420326"/>
-    <inertia ixx="0.003399" iyy="0.040399" izz="0.043145" ixy="4.2e-05" iyz="-0.0" ixz="0.0"/>
+    <origin xyz="0.2110416079169363 -0.03064586937985538 1.5515587032943756e-06" rpy="0 0 0"/>
+    <mass value="4.345058247420323"/>
+    <inertia ixx="0.003399" iyy="0.040399" izz="0.043145" ixy="-4.2e-05" iyz="0.0" ixz="-0.0"/>
   </inertial>
   <visual>
-    <origin xyz="0.382765 0.04912 0.267639" rpy="0 0 0"/>
+    <origin xyz="0.32002 -0.0308 0.303283" rpy="0 0 0"/>
     <geometry>
       <mesh filename="file://$(find surg_bot_description)/meshes/link3_1_1.stl" scale="0.001 0.001 0.001"/>
@@ -78,5 +78,5 @@
   </visual>
   <collision>
-    <origin xyz="0.382765 0.04912 0.267639" rpy="0 0 0"/>
+    <origin xyz="0.32002 -0.0308 0.303283" rpy="0 0 0"/>
     <geometry>
       <mesh filename="file://$(find surg_bot_description)/meshes/link3_1_1.stl" scale="0.001 0.001 0.001"/>
@@ -86,10 +86,10 @@
 <link name="link4_1_1">
   <inertial>
-    <origin xyz="0.029751892519794897 -0.049482100868121964 -2.921340474681955e-05" rpy="0 0 0"/>
-    <mass value="1.5005223483382892"/>
+    <origin xyz="0.027751206627339403 -0.049481985744040745 -2.8670883511938694e-05" rpy="0 0 0"/>
+    <mass value="1.50052234833829"/>
     <inertia ixx="0.00166" iyy="0.002022" izz="0.002999" ixy="0.000773" iyz="-0.0" ixz="2e-06"/>
   </inertial>
   <visual>
-    <origin xyz="-0.018748 0.01857 0.267643" rpy="0 0 0"/>
+    <origin xyz="-0.081494 -0.00025 0.30328" rpy="0 0 0"/>
     <geometry>
       <mesh filename="file://$(find surg_bot_description)/meshes/link4_1_1.stl" scale="0.001 0.001 0.001"/>
@@ -98,5 +98,5 @@
   </visual>
   <collision>
-    <origin xyz="-0.018748 0.01857 0.267643" rpy="0 0 0"/>
+    <origin xyz="-0.081494 -0.00025 0.30328" rpy="0 0 0"/>
     <geometry>
       <mesh filename="file://$(find surg_bot_description)/meshes/link4_1_1.stl" scale="0.001 0.001 0.001"/>
@@ -106,10 +106,10 @@
 <link name="link5_1_1">
   <inertial>
-    <origin xyz="3.372453495051331e-05 0.040813406687341375 0.000587414034003364" rpy="0 0 0"/>
-    <mass value="0.3856498141159764"/>
+    <origin xyz="3.305227672389943e-05 0.04081352935092518 0.0005877302186016453" rpy="0 0 0"/>
+    <mass value="0.3856498141159767"/>
     <inertia ixx="0.000311" iyy="0.000348" izz="0.000552" ixy="-0.0" iyz="-1e-06" ixz="0.0"/>
   </inertial>
   <visual>
-    <origin xyz="-0.087798 0.06892 0.267643" rpy="0 0 0"/>
+    <origin xyz="-0.148544 0.0501 0.303279" rpy="0 0 0"/>
     <geometry>
       <mesh filename="file://$(find surg_bot_description)/meshes/link5_1_1.stl" scale="0.001 0.001 0.001"/>
@@ -118,5 +118,5 @@
   </visual>
   <collision>
-    <origin xyz="-0.087798 0.06892 0.267643" rpy="0 0 0"/>
+    <origin xyz="-0.148544 0.0501 0.303279" rpy="0 0 0"/>
     <geometry>
       <mesh filename="file://$(find surg_bot_description)/meshes/link5_1_1.stl" scale="0.001 0.001 0.001"/>
@@ -126,10 +126,10 @@
 <link name="end_effector_1_1">
   <inertial>
-    <origin xyz="1.4572522974432012e-07 -1.2266364841223565e-07 -0.0025003780571151712" rpy="0 0 0"/>
+    <origin xyz="-1.822417527441722e-07 6.200430793801281e-13 -0.002500062517189483" rpy="0 0 0"/>
     <mass value="0.001098697673021953"/>
-    <inertia ixx="0.0" iyy="0.0" izz="0.0" ixy="0.0" iyz="0.0" ixz="0.0"/>
+    <inertia ixx="0.0" iyy="0.0" izz="0.0" ixy="-0.0" iyz="-0.0" ixz="-0.0"/>
   </inertial>
   <visual>
-    <origin xyz="-0.087798 0.02552 0.282393" rpy="0 0 0"/>
+    <origin xyz="-0.148544 0.0067 0.318029" rpy="0 0 0"/>
     <geometry>
       <mesh filename="file://$(find surg_bot_description)/meshes/end_effector_1_1.stl" scale="0.001 0.001 0.001"/>
@@ -138,5 +138,5 @@
   </visual>
   <collision>
-    <origin xyz="-0.087798 0.02552 0.282393" rpy="0 0 0"/>
+    <origin xyz="-0.148544 0.0067 0.318029" rpy="0 0 0"/>
     <geometry>
       <mesh filename="file://$(find surg_bot_description)/meshes/end_effector_1_1.stl" scale="0.001 0.001 0.001"/>
@@ -144,11 +144,11 @@
   </collision>
 </link>
-<joint name="Revolute 7" type="continuous">
-  <origin xyz="-0.062755 -0.01851 -0.028139" rpy="0 0 0"/>
+<joint name="Revolute 1" type="continuous">
+  <origin xyz="-1e-05 1e-05 -0.063784" rpy="0 0 0"/>
   <parent link="base_link"/>
   <child link="link1_1_1"/>
-  <axis xyz="-0.0 0.0 1.0"/>
+  <axis xyz="0.0 0.0 1.0"/>
 </joint>
-<joint name="Revolute 8" type="continuous">
+<joint name="Revolute2" type="continuous">
   <origin xyz="-0.32002 0.0 -0.035216" rpy="0 0 0"/>
   <parent link="link1_1_1"/>
@@ -156,20 +156,20 @@
   <axis xyz="0.0 0.0 1.0"/>
 </joint>
-<joint name="Revolute 9" type="revolute">
-  <origin xyz="1e-05 -0.03061 -0.204284" rpy="0 0 0"/>
+<joint name="Revolute 3" type="revolute">
+  <origin xyz="1e-05 0.03079 -0.204283" rpy="0 0 0"/>
   <parent link="link2_1_1"/>
   <child link="link3_1_1"/>
-  <axis xyz="0.0 -1.0 0.0"/>
-  <limit upper="0.174533" lower="-1.570796" effort="100" velocity="100"/>
+  <axis xyz="0.0 1.0 -0.0"/>
+  <limit upper="1.570796" lower="-0.174533" effort="100" velocity="100"/>
 </joint>
-<joint name="Revolute 10" type="revolute">
-  <origin xyz="0.401513 0.03055 -4e-06" rpy="0 0 0"/>
+<joint name="Revolute 4" type="revolute">
+  <origin xyz="0.401514 -0.03055 3e-06" rpy="0 0 0"/>
   <parent link="link3_1_1"/>
   <child link="link4_1_1"/>
-  <axis xyz="1.0 -0.0 -1e-05"/>
+  <axis xyz="1.0 0.0 1e-05"/>
   <limit upper="2.268928" lower="-2.268928" effort="100" velocity="100"/>
 </joint>
-<joint name="Revolute 11" type="revolute">
-  <origin xyz="0.06905 -0.05035 0.0" rpy="0 0 0"/>
+<joint name="Revolute 5" type="revolute">
+  <origin xyz="0.06705 -0.05035 1e-06" rpy="0 0 0"/>
   <parent link="link4_1_1"/>
   <child link="link5_1_1"/>
@@ -177,5 +177,5 @@
   <limit upper="2.268928" lower="-2.268928" effort="100" velocity="100"/>
 </joint>
-<joint name="Rigid 12" type="fixed">
+<joint name="Rigid 1" type="fixed">
   <origin xyz="0.0 0.0434 -0.01475" rpy="0 0 0"/>
   <parent link="link5_1_1"/>

Commit message: Fixed all description and config files

File: ros2_ws/src/surg_bot_description/urdf/surg_bot.xacro (robot description, xacro)
@@ -150,5 +150,5 @@
   <axis xyz="0.0 0.0 1.0"/>
 </joint>
-<joint name="Revolute2" type="continuous">
+<joint name="Revolute 2" type="continuous">
   <origin xyz="-0.32002 0.0 -0.035216" rpy="0 0 0"/>
   <parent link="link1_1_1"/>
