Commit message: Refactor joint names to lowercase and update related configurations for consistency

File: ros2_ws/src/surg_bot_description/urdf/surg_bot.xacro (robot description, xacro)
@@ -144,5 +144,5 @@
   </collision>
 </link>
-<joint name="Revolute 1" type="continuous">
+<joint name="revolute_1" type="continuous">
   <origin xyz="-1e-05 1e-05 -0.063784" rpy="0 0 0"/>
   <parent link="base_link"/>
@@ -150,5 +150,5 @@
   <axis xyz="0.0 0.0 1.0"/>
 </joint>
-<joint name="Revolute 2" type="continuous">
+<joint name="revolute_2" type="continuous">
   <origin xyz="-0.32002 0.0 -0.035216" rpy="0 0 0"/>
   <parent link="link1_1_1"/>
@@ -156,5 +156,5 @@
   <axis xyz="0.0 0.0 1.0"/>
 </joint>
-<joint name="Revolute 3" type="revolute">
+<joint name="revolute_3" type="revolute">
   <origin xyz="1e-05 0.03079 -0.204283" rpy="0 0 0"/>
   <parent link="link2_1_1"/>
@@ -163,5 +163,5 @@
   <limit upper="1.570796" lower="-0.174533" effort="100" velocity="100"/>
 </joint>
-<joint name="Revolute 4" type="revolute">
+<joint name="revolute_4" type="revolute">
   <origin xyz="0.401514 -0.03055 3e-06" rpy="0 0 0"/>
   <parent link="link3_1_1"/>
@@ -170,5 +170,5 @@
   <limit upper="2.268928" lower="-2.268928" effort="100" velocity="100"/>
 </joint>
-<joint name="Revolute 5" type="revolute">
+<joint name="revolute_5" type="revolute">
   <origin xyz="0.06705 -0.05035 1e-06" rpy="0 0 0"/>
   <parent link="link4_1_1"/>
@@ -177,5 +177,5 @@
   <limit upper="2.268928" lower="-2.268928" effort="100" velocity="100"/>
 </joint>
-<joint name="Rigid 1" type="fixed">
+<joint name="rigid_1" type="fixed">
   <origin xyz="0.0 0.0434 -0.01475" rpy="0 0 0"/>
   <parent link="link5_1_1"/>

File: ros2_ws/src/surg_bot_moveit_config/config/surg_bot.ros2_control.xacro (robot description, xacro)
@@ -8,32 +8,32 @@
                 <plugin>mock_components/GenericSystem</plugin>
             </hardware>
-            <joint name="Revolute 1">
+            <joint name="revolute_1">
                 <command_interface name="position"/>
                 <state_interface name="position">
-                  <param name="initial_value">${initial_positions['Revolute 1']}</param>
+                  <param name="initial_value">${initial_positions['revolute_1']}</param>
                 </state_interface>
             </joint>
-            <joint name="Revolute 2">
+            <joint name="revolute_2">
                 <command_interface name="position"/>
                 <state_interface name="position">
-                  <param name="initial_value">${initial_positions['Revolute 2']}</param>
+                  <param name="initial_value">${initial_positions['revolute_2']}</param>
                 </state_interface>
             </joint>
-            <joint name="Revolute 3">
+            <joint name="revolute_3">
                 <command_interface name="position"/>
                 <state_interface name="position">
-                  <param name="initial_value">${initial_positions['Revolute 3']}</param>
+                  <param name="initial_value">${initial_positions['revolute_3']}</param>
                 </state_interface>
             </joint>
-            <joint name="Revolute 4">
+            <joint name="revolute_4">
                 <command_interface name="position"/>
                 <state_interface name="position">
-                  <param name="initial_value">${initial_positions['Revolute 4']}</param>
+                  <param name="initial_value">${initial_positions['revolute_4']}</param>
                 </state_interface>
             </joint>
-            <joint name="Revolute 5">
+            <joint name="revolute_5">
                 <command_interface name="position"/>
                 <state_interface name="position">
-                  <param name="initial_value">${initial_positions['Revolute 5']}</param>
+                  <param name="initial_value">${initial_positions['revolute_5']}</param>
                 </state_interface>
             </joint>

Commit message: Fix URDF for shorter link3

File: ros2_ws/src/surg_bot_description/urdf/surg_bot.xacro (robot description, xacro)
@@ -26,7 +26,7 @@
 <link name="link1_1_1">
   <inertial>
-    <origin xyz="-0.16001007717101118 -1.5433885539871676e-05 -0.01760775000004905" rpy="0 0 0"/>
+    <origin xyz="-0.16000855446108672 0.0006982755267684382 -0.017607750000049494" rpy="0 0 0"/>
     <mass value="8.367890341080868"/>
-    <inertia ixx="0.012225" iyy="0.118361" izz="0.124365" ixy="0.0" iyz="0.0" ixz="0.001924"/>
+    <inertia ixx="0.012227" iyy="0.118359" izz="0.124365" ixy="0.000473" iyz="-9e-06" ixz="0.001924"/>
   </inertial>
   <visual>
@@ -46,10 +46,10 @@
 <link name="link2_1_1">
   <inertial>
-    <origin xyz="0.00022218321954753373 2.5577962440391797e-05 -0.11737411773568335" rpy="0 0 0"/>
+    <origin xyz="0.0002224902754690561 2.4896581295632018e-05 -0.1173741177356834" rpy="0 0 0"/>
     <mass value="3.3490679501648595"/>
-    <inertia ixx="0.014417" iyy="0.014057" izz="0.002264" ixy="0.0" iyz="8e-06" ixz="-5.7e-05"/>
+    <inertia ixx="0.014417" iyy="0.014057" izz="0.002264" ixy="-2e-06" iyz="8e-06" ixz="-5.7e-05"/>
   </inertial>
   <visual>
-    <origin xyz="0.32003 -1e-05 0.099" rpy="0 0 0"/>
+    <origin xyz="0.320027 -0.001437 0.099" rpy="0 0 0"/>
     <geometry>
       <mesh filename="file://$(find surg_bot_description)/meshes/link2_1_1.stl" scale="0.001 0.001 0.001"/>
@@ -58,5 +58,5 @@
   </visual>
   <collision>
-    <origin xyz="0.32003 -1e-05 0.099" rpy="0 0 0"/>
+    <origin xyz="0.320027 -0.001437 0.099" rpy="0 0 0"/>
     <geometry>
       <mesh filename="file://$(find surg_bot_description)/meshes/link2_1_1.stl" scale="0.001 0.001 0.001"/>
@@ -64,41 +64,41 @@
   </collision>
 </link>
-<link name="link3_1_1">
+<link name="link3_1">
   <inertial>
-    <origin xyz="0.2110416079169363 -0.03064586937985538 1.5515587032943756e-06" rpy="0 0 0"/>
-    <mass value="4.345058247420323"/>
-    <inertia ixx="0.003399" iyy="0.040399" izz="0.043145" ixy="-4.2e-05" iyz="0.0" ixz="-0.0"/>
+    <origin xyz="0.13549556866217186 0.030032525454134127 -4.999999703714231e-07" rpy="0 0 0"/>
+    <mass value="1.7602626049739658"/>
+    <inertia ixx="0.001766" iyy="0.008244" izz="0.009744" ixy="3.2e-05" iyz="0.0" ixz="0.0"/>
   </inertial>
   <visual>
-    <origin xyz="0.32002 -0.0308 0.303283" rpy="0 0 0"/>
+    <origin xyz="0.320168 0.029172 0.303283" rpy="0 0 0"/>
     <geometry>
-      <mesh filename="file://$(find surg_bot_description)/meshes/link3_1_1.stl" scale="0.001 0.001 0.001"/>
+      <mesh filename="file://$(find surg_bot_description)/meshes/link3_1.stl" scale="0.001 0.001 0.001"/>
     </geometry>
     <material name="silver"/>
   </visual>
   <collision>
-    <origin xyz="0.32002 -0.0308 0.303283" rpy="0 0 0"/>
+    <origin xyz="0.320168 0.029172 0.303283" rpy="0 0 0"/>
     <geometry>
-      <mesh filename="file://$(find surg_bot_description)/meshes/link3_1_1.stl" scale="0.001 0.001 0.001"/>
+      <mesh filename="file://$(find surg_bot_description)/meshes/link3_1.stl" scale="0.001 0.001 0.001"/>
     </geometry>
   </collision>
 </link>
-<link name="link4_1_1">
+<link name="link4_1">
   <inertial>
-    <origin xyz="0.027751206627339403 -0.049481985744040745 -2.8670883511938694e-05" rpy="0 0 0"/>
-    <mass value="1.50052234833829"/>
-    <inertia ixx="0.00166" iyy="0.002022" izz="0.002999" ixy="0.000773" iyz="-0.0" ixz="2e-06"/>
+    <origin xyz="0.02600502860609198 -0.04510246183047751 -5.119758128557805e-07" rpy="0 0 0"/>
+    <mass value="1.4039319321687402"/>
+    <inertia ixx="0.00142" iyy="0.001886" izz="0.002652" ixy="0.000674" iyz="0.0" ixz="-0.0"/>
   </inertial>
   <visual>
-    <origin xyz="-0.081494 -0.00025 0.30328" rpy="0 0 0"/>
+    <origin xyz="0.065316 -0.000267 0.303283" rpy="0 0 0"/>
     <geometry>
-      <mesh filename="file://$(find surg_bot_description)/meshes/link4_1_1.stl" scale="0.001 0.001 0.001"/>
+      <mesh filename="file://$(find surg_bot_description)/meshes/link4_1.stl" scale="0.001 0.001 0.001"/>
     </geometry>
     <material name="silver"/>
   </visual>
   <collision>
-    <origin xyz="-0.081494 -0.00025 0.30328" rpy="0 0 0"/>
+    <origin xyz="0.065316 -0.000267 0.303283" rpy="0 0 0"/>
     <geometry>
-      <mesh filename="file://$(find surg_bot_description)/meshes/link4_1_1.stl" scale="0.001 0.001 0.001"/>
+      <mesh filename="file://$(find surg_bot_description)/meshes/link4_1.stl" scale="0.001 0.001 0.001"/>
     </geometry>
   </collision>
@@ -106,10 +106,10 @@
 <link name="link5_1_1">
   <inertial>
-    <origin xyz="3.305227672389943e-05 0.04081352935092518 0.0005877302186016453" rpy="0 0 0"/>
-    <mass value="0.3856498141159767"/>
-    <inertia ixx="0.000311" iyy="0.000348" izz="0.000552" ixy="-0.0" iyz="-1e-06" ixz="0.0"/>
+    <origin xyz="0.0002259892794144409 0.03886333123442502 0.0005887467592404771" rpy="0 0 0"/>
+    <mass value="0.38469776659589416"/>
+    <inertia ixx="0.000309" iyy="0.000348" izz="0.00055" ixy="0.0" iyz="-1e-06" ixz="0.0"/>
   </inertial>
   <visual>
-    <origin xyz="-0.148544 0.0501 0.303279" rpy="0 0 0"/>
+    <origin xyz="0.000274 0.041925 0.303283" rpy="0 0 0"/>
     <geometry>
       <mesh filename="file://$(find surg_bot_description)/meshes/link5_1_1.stl" scale="0.001 0.001 0.001"/>
@@ -118,5 +118,5 @@
   </visual>
   <collision>
-    <origin xyz="-0.148544 0.0501 0.303279" rpy="0 0 0"/>
+    <origin xyz="0.000274 0.041925 0.303283" rpy="0 0 0"/>
     <geometry>
       <mesh filename="file://$(find surg_bot_description)/meshes/link5_1_1.stl" scale="0.001 0.001 0.001"/>
@@ -126,10 +126,10 @@
 <link name="end_effector_1_1">
   <inertial>
-    <origin xyz="-1.822417527441722e-07 6.200430793801281e-13 -0.002500062517189483" rpy="0 0 0"/>
+    <origin xyz="-2.7668857425572823e-07 -2.5305395503594057e-07 0.002499500002298649" rpy="0 0 0"/>
     <mass value="0.001098697673021953"/>
-    <inertia ixx="0.0" iyy="0.0" izz="0.0" ixy="-0.0" iyz="-0.0" ixz="-0.0"/>
+    <inertia ixx="0.0" iyy="0.0" izz="0.0" ixy="-0.0" iyz="-0.0" ixz="0.0"/>
   </inertial>
   <visual>
-    <origin xyz="-0.148544 0.0067 0.318029" rpy="0 0 0"/>
+    <origin xyz="6.9e-05 0.000575 0.318033" rpy="0 0 0"/>
     <geometry>
       <mesh filename="file://$(find surg_bot_description)/meshes/end_effector_1_1.stl" scale="0.001 0.001 0.001"/>
@@ -138,5 +138,5 @@
   </visual>
   <collision>
-    <origin xyz="-0.148544 0.0067 0.318029" rpy="0 0 0"/>
+    <origin xyz="6.9e-05 0.000575 0.318033" rpy="0 0 0"/>
     <geometry>
       <mesh filename="file://$(find surg_bot_description)/meshes/end_effector_1_1.stl" scale="0.001 0.001 0.001"/>
@@ -144,5 +144,5 @@
   </collision>
 </link>
-<joint name="revolute_1" type="continuous">
+<joint name="joint0" type="continuous">
   <origin xyz="-1e-05 1e-05 -0.063784" rpy="0 0 0"/>
   <parent link="base_link"/>
@@ -150,33 +150,32 @@
   <axis xyz="0.0 0.0 1.0"/>
 </joint>
-<joint name="revolute_2" type="continuous">
-  <origin xyz="-0.32002 0.0 -0.035216" rpy="0 0 0"/>
+<joint name="joint1" type="continuous">
+  <origin xyz="-0.320017 0.001427 -0.035216" rpy="0 0 0"/>
   <parent link="link1_1_1"/>
   <child link="link2_1_1"/>
   <axis xyz="0.0 0.0 1.0"/>
 </joint>
-<joint name="revolute_3" type="revolute">
-  <origin xyz="1e-05 0.03079 -0.204283" rpy="0 0 0"/>
+<joint name="joint2" type="revolute">
+  <origin xyz="-0.000141 -0.030609 -0.204283" rpy="0 0 0"/>
   <parent link="link2_1_1"/>
-  <child link="link3_1_1"/>
-  <axis xyz="0.0 1.0 -0.0"/>
-  <limit upper="1.570796" lower="-0.174533" effort="100" velocity="100"/>
+  <child link="link3_1"/>
+  <axis xyz="-0.004946 -0.999988 0.0"/>
+  <limit upper="0.174533" lower="-1.570796" effort="100" velocity="100"/>
 </joint>
-<joint name="revolute_4" type="revolute">
-  <origin xyz="0.401514 -0.03055 3e-06" rpy="0 0 0"/>
-  <parent link="link3_1_1"/>
-  <child link="link4_1_1"/>
-  <axis xyz="1.0 0.0 1e-05"/>
+<joint name="joint3" type="revolute">
+  <origin xyz="0.254852 0.029439 0.0" rpy="0 0 0"/>
+  <parent link="link3_1"/>
+  <child link="link4_1"/>
+  <axis xyz="0.999988 -0.004946 0.0"/>
   <limit upper="2.268928" lower="-2.268928" effort="100" velocity="100"/>
 </joint>
-<joint name="revolute_5" type="revolute">
-  <origin xyz="0.06705 -0.05035 1e-06" rpy="0 0 0"/>
-  <parent link="link4_1_1"/>
+<joint name="joint4" type="continuous">
+  <origin xyz="0.065042 -0.042192 0.0" rpy="0 0 0"/>
+  <parent link="link4_1"/>
   <child link="link5_1_1"/>
-  <axis xyz="0.0 1.0 0.0"/>
-  <limit upper="2.268928" lower="-2.268928" effort="100" velocity="100"/>
+  <axis xyz="0.004946 0.999988 -0.0"/>
 </joint>
-<joint name="rigid_1" type="fixed">
-  <origin xyz="0.0 0.0434 -0.01475" rpy="0 0 0"/>
+<joint name="rigid1" type="fixed">
+  <origin xyz="0.000205 0.04135 -0.01475" rpy="0 0 0"/>
   <parent link="link5_1_1"/>
   <child link="end_effector_1_1"/>

File: ros2_ws/src/surg_bot_moveit_config/config/surg_bot.ros2_control.xacro (robot description, xacro)
@@ -8,32 +8,32 @@
                 <plugin>mock_components/GenericSystem</plugin>
             </hardware>
-            <joint name="revolute_1">
+            <joint name="joint0">
                 <command_interface name="position"/>
                 <state_interface name="position">
-                  <param name="initial_value">${initial_positions['revolute_1']}</param>
+                  <param name="initial_value">${initial_positions['joint0']}</param>
                 </state_interface>
             </joint>
-            <joint name="revolute_2">
+            <joint name="joint1">
                 <command_interface name="position"/>
                 <state_interface name="position">
-                  <param name="initial_value">${initial_positions['revolute_2']}</param>
+                  <param name="initial_value">${initial_positions['joint1']}</param>
                 </state_interface>
             </joint>
-            <joint name="revolute_3">
+            <joint name="joint2">
                 <command_interface name="position"/>
                 <state_interface name="position">
-                  <param name="initial_value">${initial_positions['revolute_3']}</param>
+                  <param name="initial_value">${initial_positions['joint2']}</param>
                 </state_interface>
             </joint>
-            <joint name="revolute_4">
+            <joint name="joint3">
                 <command_interface name="position"/>
                 <state_interface name="position">
-                  <param name="initial_value">${initial_positions['revolute_4']}</param>
+                  <param name="initial_value">${initial_positions['joint3']}</param>
                 </state_interface>
             </joint>
-            <joint name="revolute_5">
+            <joint name="joint4">
                 <command_interface name="position"/>
                 <state_interface name="position">
-                  <param name="initial_value">${initial_positions['revolute_5']}</param>
+                  <param name="initial_value">${initial_positions['joint4']}</param>
                 </state_interface>
             </joint>
