Commit message: Got all the IK working, just need to do the execution

File: ros2_ws/src/surg_bot_description/urdf/surg_bot.xacro (robot description, xacro)
@@ -26,7 +26,7 @@
 <link name="link1_1_1">
   <inertial>
-    <origin xyz="-0.16000855446108672 0.0006982755267684382 -0.017607750000049494" rpy="0 0 0"/>
+    <origin xyz="-0.16001007717101143 -1.5433885540422345e-05 -0.01760775000004948" rpy="0 0 0"/>
     <mass value="8.367890341080868"/>
-    <inertia ixx="0.012227" iyy="0.118359" izz="0.124365" ixy="0.000473" iyz="-9e-06" ixz="0.001924"/>
+    <inertia ixx="0.012225" iyy="0.118361" izz="0.124365" ixy="0.0" iyz="0.0" ixz="0.001924"/>
   </inertial>
   <visual>
@@ -46,10 +46,10 @@
 <link name="link2_1_1">
   <inertial>
-    <origin xyz="0.0002224902754690561 2.4896581295632018e-05 -0.1173741177356834" rpy="0 0 0"/>
+    <origin xyz="0.00022227782028544363 2.474064107253927e-05 -0.1173741177356839" rpy="0 0 0"/>
     <mass value="3.3490679501648595"/>
-    <inertia ixx="0.014417" iyy="0.014057" izz="0.002264" ixy="-2e-06" iyz="8e-06" ixz="-5.7e-05"/>
+    <inertia ixx="0.014417" iyy="0.014057" izz="0.002264" ixy="-1e-06" iyz="8e-06" ixz="-5.7e-05"/>
   </inertial>
   <visual>
-    <origin xyz="0.320027 -0.001437 0.099" rpy="0 0 0"/>
+    <origin xyz="0.32003 -1e-05 0.099" rpy="0 0 0"/>
     <geometry>
       <mesh filename="file://$(find surg_bot_description)/meshes/link2_1_1.stl" scale="0.001 0.001 0.001"/>
@@ -58,5 +58,5 @@
   </visual>
   <collision>
-    <origin xyz="0.320027 -0.001437 0.099" rpy="0 0 0"/>
+    <origin xyz="0.32003 -1e-05 0.099" rpy="0 0 0"/>
     <geometry>
       <mesh filename="file://$(find surg_bot_description)/meshes/link2_1_1.stl" scale="0.001 0.001 0.001"/>
@@ -66,10 +66,10 @@
 <link name="link3_1">
   <inertial>
-    <origin xyz="0.13549556866217186 0.030032525454134127 -4.999999703714231e-07" rpy="0 0 0"/>
+    <origin xyz="0.13545922670739144 0.030192910577609006 0.00044866468088849976" rpy="0 0 0"/>
     <mass value="1.7602626049739658"/>
-    <inertia ixx="0.001766" iyy="0.008244" izz="0.009744" ixy="3.2e-05" iyz="0.0" ixz="0.0"/>
+    <inertia ixx="0.001766" iyy="0.008244" izz="0.009744" ixy="2.4e-05" iyz="0.0" ixz="-2.6e-05"/>
   </inertial>
   <visual>
-    <origin xyz="0.320168 0.029172 0.303283" rpy="0 0 0"/>
+    <origin xyz="0.320135 0.0306 0.303283" rpy="0 0 0"/>
     <geometry>
       <mesh filename="file://$(find surg_bot_description)/meshes/link3_1.stl" scale="0.001 0.001 0.001"/>
@@ -78,5 +78,5 @@
   </visual>
   <collision>
-    <origin xyz="0.320168 0.029172 0.303283" rpy="0 0 0"/>
+    <origin xyz="0.320135 0.0306 0.303283" rpy="0 0 0"/>
     <geometry>
       <mesh filename="file://$(find surg_bot_description)/meshes/link3_1.stl" scale="0.001 0.001 0.001"/>
@@ -86,10 +86,10 @@
 <link name="link4_1">
   <inertial>
-    <origin xyz="0.02600502860609198 -0.04510246183047751 -5.119758128557805e-07" rpy="0 0 0"/>
+    <origin xyz="0.02605773282976529 -0.04507242712799745 8.675535075214347e-05" rpy="0 0 0"/>
     <mass value="1.4039319321687402"/>
-    <inertia ixx="0.00142" iyy="0.001886" izz="0.002652" ixy="0.000674" iyz="0.0" ixz="-0.0"/>
+    <inertia ixx="0.001418" iyy="0.001888" izz="0.002652" ixy="0.000674" iyz="2e-06" ixz="-4e-06"/>
   </inertial>
   <visual>
-    <origin xyz="0.065316 -0.000267 0.303283" rpy="0 0 0"/>
+    <origin xyz="0.065319 0.000859 0.302438" rpy="0 0 0"/>
     <geometry>
       <mesh filename="file://$(find surg_bot_description)/meshes/link4_1.stl" scale="0.001 0.001 0.001"/>
@@ -98,5 +98,5 @@
   </visual>
   <collision>
-    <origin xyz="0.065316 -0.000267 0.303283" rpy="0 0 0"/>
+    <origin xyz="0.065319 0.000859 0.302438" rpy="0 0 0"/>
     <geometry>
       <mesh filename="file://$(find surg_bot_description)/meshes/link4_1.stl" scale="0.001 0.001 0.001"/>
@@ -106,10 +106,10 @@
 <link name="link5_1_1">
   <inertial>
-    <origin xyz="0.0002259892794144409 0.03886333123442502 0.0005887467592404771" rpy="0 0 0"/>
+    <origin xyz="0.0001801099222721872 0.03886369124244137 0.0005895595584266555" rpy="0 0 0"/>
     <mass value="0.38469776659589416"/>
     <inertia ixx="0.000309" iyy="0.000348" izz="0.00055" ixy="0.0" iyz="-1e-06" ixz="0.0"/>
   </inertial>
   <visual>
-    <origin xyz="0.000274 0.041925 0.303283" rpy="0 0 0"/>
+    <origin xyz="0.000228 0.042975 0.302222" rpy="0 0 0"/>
     <geometry>
       <mesh filename="file://$(find surg_bot_description)/meshes/link5_1_1.stl" scale="0.001 0.001 0.001"/>
@@ -118,5 +118,5 @@
   </visual>
   <collision>
-    <origin xyz="0.000274 0.041925 0.303283" rpy="0 0 0"/>
+    <origin xyz="0.000228 0.042975 0.302222" rpy="0 0 0"/>
     <geometry>
       <mesh filename="file://$(find surg_bot_description)/meshes/link5_1_1.stl" scale="0.001 0.001 0.001"/>
@@ -126,10 +126,10 @@
 <link name="end_effector_1_1">
   <inertial>
-    <origin xyz="-2.7668857425572823e-07 -2.5305395503594057e-07 0.002499500002298649" rpy="0 0 0"/>
+    <origin xyz="4.038171408361996e-07 9.114467316127806e-08 0.0025003140135481106" rpy="0 0 0"/>
     <mass value="0.001098697673021953"/>
-    <inertia ixx="0.0" iyy="0.0" izz="0.0" ixy="-0.0" iyz="-0.0" ixz="0.0"/>
+    <inertia ixx="0.0" iyy="0.0" izz="0.0" ixy="0.0" iyz="-0.0" ixz="-0.0"/>
   </inertial>
   <visual>
-    <origin xyz="6.9e-05 0.000575 0.318033" rpy="0 0 0"/>
+    <origin xyz="7.2e-05 0.001625 0.316972" rpy="0 0 0"/>
     <geometry>
       <mesh filename="file://$(find surg_bot_description)/meshes/end_effector_1_1.stl" scale="0.001 0.001 0.001"/>
@@ -138,5 +138,5 @@
   </visual>
   <collision>
-    <origin xyz="6.9e-05 0.000575 0.318033" rpy="0 0 0"/>
+    <origin xyz="7.2e-05 0.001625 0.316972" rpy="0 0 0"/>
     <geometry>
       <mesh filename="file://$(find surg_bot_description)/meshes/end_effector_1_1.stl" scale="0.001 0.001 0.001"/>
@@ -144,40 +144,45 @@
   </collision>
 </link>
-<joint name="joint0" type="continuous">
+<joint name="joint0" type="revolute">
   <origin xyz="-1e-05 1e-05 -0.063784" rpy="0 0 0"/>
   <parent link="base_link"/>
   <child link="link1_1_1"/>
   <axis xyz="0.0 0.0 1.0"/>
+  <limit upper="3.141593" lower="-3.141593" effort="100" velocity="100"/>
 </joint>
-<joint name="joint1" type="continuous">
-  <origin xyz="-0.320017 0.001427 -0.035216" rpy="0 0 0"/>
+<joint name="joint1" type="revolute">
+  <origin xyz="-0.32002 0.0 -0.035216" rpy="0 0 0"/>
   <parent link="link1_1_1"/>
   <child link="link2_1_1"/>
   <axis xyz="0.0 0.0 1.0"/>
+  <limit upper="3.141593" lower="-3.141593" effort="100" velocity="100"/>
 </joint>
 <joint name="joint2" type="revolute">
-  <origin xyz="-0.000141 -0.030609 -0.204283" rpy="0 0 0"/>
+  <origin xyz="-0.000105 -0.03061 -0.204283" rpy="0 0 0"/>
   <parent link="link2_1_1"/>
   <child link="link3_1"/>
-  <axis xyz="-0.004946 -0.999988 0.0"/>
+  <axis xyz="-0.003766 -0.999993 0.0"/>
   <limit upper="0.174533" lower="-1.570796" effort="100" velocity="100"/>
 </joint>
 <joint name="joint3" type="revolute">
-  <origin xyz="0.254852 0.029439 0.0" rpy="0 0 0"/>
+  <origin xyz="0.254816 0.029741 0.000845" rpy="0 0 0"/>
   <parent link="link3_1"/>
   <child link="link4_1"/>
-  <axis xyz="0.999988 -0.004946 0.0"/>
+  <axis xyz="0.999987 -0.003766 0.003319"/>
   <limit upper="2.268928" lower="-2.268928" effort="100" velocity="100"/>
 </joint>
-<joint name="joint4" type="continuous">
-  <origin xyz="0.065042 -0.042192 0.0" rpy="0 0 0"/>
+<joint name="joint4" type="revolute">
+  <origin xyz="0.065091 -0.042116 0.000216" rpy="0 0 0"/>
   <parent link="link4_1"/>
   <child link="link5_1_1"/>
-  <axis xyz="0.004946 0.999988 -0.0"/>
+  <axis xyz="0.003766 0.999993 1e-06"/>
+  <limit upper="2.268928" lower="-2.268928" effort="100" velocity="100"/>
 </joint>
-<joint name="rigid1" type="fixed">
-  <origin xyz="0.000205 0.04135 -0.01475" rpy="0 0 0"/>
+<joint name="joint5" type="revolute">
+  <origin xyz="0.000156 0.04135 -0.01475" rpy="0 0 0"/>
   <parent link="link5_1_1"/>
   <child link="end_effector_1_1"/>
+  <axis xyz="1.9e-05 1e-06 -1.0"/>
+  <limit upper="3.141593" lower="-3.141593" effort="100" velocity="100"/>
 </joint>
 </robot>

File: ros2_ws/src/surg_bot_moveit_config/config/surg_bot.ros2_control.xacro (robot description, xacro)
@@ -38,4 +38,10 @@
                 </state_interface>
             </joint>
+            <joint name="joint5">
+                <command_interface name="position"/>
+                <state_interface name="position">
+                  <param name="initial_value">${initial_positions['joint5']}</param>
+                </state_interface>
+            </joint>
         </ros2_control>
     </xacro:macro>
